File: pcb/ZeroPCB.sch (KiCad schematic (older format))
At the start: 0 parts

Commit message: Finish the schematic
Changed lines of the file:
@@
 $Descr A4 11693 8268
 encoding utf-8
-Sheet 1 5
+Sheet 1 8
 Title ""
 Date ""
@@
 $EndDescr
 $Sheet
-S 2100 1650 1400 1150
+S 4400 1400 1400 750
 U 612A12A2
 F0 "power" 50
 F1 "power.sch" 50
-F2 "BAT_REF" O R 3500 2300 50
-F3 "1.65V" O R 3500 2500 50
-$EndSheet
-$Sheet
-S 2600 3700 1600 650
+F2 "BAT_REF" O R 5800 1650 50
+F3 "1.65V" O L 4400 2050 50
+$EndSheet
+$Sheet
+S 4100 3800 1700 600
+U 613586C8
+F0 "Motor" 50
+F1 "Motor.sch" 50
+F2 "Left_EncoderA" O R 5800 3950 50
+F3 "Left_EncoderB" O R 5800 4050 50
+F4 "Right_EncoderA" O R 5800 4200 50
+F5 "Right_EncoderB" O R 5800 4300 50
+F6 "Left_Motor_OUT1" I L 4100 3950 50
+F7 "Left_Motor_OUT2" I L 4100 4050 50
+F8 "Right_Motor_OUT1" I L 4100 4200 50
+F9 "Right_Motor_OUT2" I L 4100 4300 50
+$EndSheet
+$Sheet
+S 9000 2450 550  800
+U 6169318F
+F0 "Communication" 50
+F1 "Communication.sch" 50
+F2 "UART_TX" I L 9000 2650 50
+F3 "UART_RX" O L 9000 2750 50
+F4 "SWCLK" I L 9000 2950 50
+F5 "SWDIO" B L 9000 3050 50
+F6 "NRST" O L 9000 3150 50
+$EndSheet
+Wire Wire Line
+	7850 2150 9000 2150
+Wire Wire Line
+	7850 2050 9000 2050
+Wire Wire Line
+	7850 1950 9000 1950
+Wire Wire Line
+	7850 1850 9000 1850
+Wire Wire Line
+	7850 1750 9000 1750
+Wire Wire Line
+	7850 1650 9000 1650
+$Sheet
+S 9000 1400 550  850
+U 61682BF7
+F0 "Debug" 50
+F1 "Debug.sch" 50
+F2 "LED1" I L 9000 1650 50
+F3 "LED2" I L 9000 1750 50
+F4 "LED3" I L 9000 1850 50
+F5 "LED4" I L 9000 1950 50
+F6 "LED5" I L 9000 2050 50
+F7 "Buzzer" I L 9000 1500 50
+F8 "LED6" I L 9000 2150 50
+$EndSheet
+Wire Wire Line
+	4400 2050 4150 2050
+$Sheet
+S 8100 3700 700  850
+U 6163ECBF
+F0 "GyroSensor" 50
+F1 "GyroSensor.sch" 50
+F2 "IMU_MOSI" I L 8100 4000 50
+F3 "IMU_MISO" O L 8100 4250 50
+F4 "IMU_CLK" I L 8100 3850 50
+F5 "IMU_CS" I L 8100 4400 50
+$EndSheet
+Wire Wire Line
+	9000 2750 7850 2750
+Wire Wire Line
+	7850 2650 9000 2650
+Wire Wire Line
+	7850 3850 8100 3850
+Wire Wire Line
+	7850 4000 8100 4000
+Wire Wire Line
+	7850 4250 8100 4250
+Wire Wire Line
+	7850 4400 8100 4400
+Wire Wire Line
+	7850 2950 9000 2950
+Wire Wire Line
+	7850 3150 9000 3150
+Wire Wire Line
+	9000 3050 7850 3050
+Wire Wire Line
+	5800 1650 6450 1650
+$Sheet
+S 4400 2350 1400 900
 U 6135359E
 F0 "IRSensor" 50
 F1 "IRSensor.sch" 50
-F2 "IR_Sensor_OUT1" I L 2600 4000 50
-F3 "IR_Sensor_OUT2" I L 2600 4100 50
-F4 "1.65V" I L 2600 3900 50
-F5 "IR_Sensor_IN1" O R 4200 3900 50
-F6 "IR_Sensor_IN2" O R 4200 4000 50
-F7 "IR_Sensor_IN3" O R 4200 4100 50
-F8 "IR_Sensor_IN4" O R 4200 4200 50
-$EndSheet
-Wire Wire Line
-	2600 3900 2250 3900
-Wire Wire Line
-	2250 3900 2250 3050
-Wire Wire Line
-	2250 3050 3800 3050
-Wire Wire Line
-	3800 3050 3800 2500
-Wire Wire Line
-	3800 2500 3500 2500
-$Sheet
-S 2050 5050 1700 600
-U 613586C8
-F0 "Motor" 50
-F1 "Motor.sch" 50
-F2 "Left_Encoder_A" O R 3750 5200 50
-F3 "Left_Encoder_B" O R 3750 5300 50
-F4 "Right_Encoder_A" O R 3750 5400 50
-F5 "Right_Encoder_B" O R 3750 5500 50
-F6 "Left_Motor_OUT_A" I L 2050 5200 50
-F7 "Left_Motor_OUT_B" I L 2050 5300 50
-F8 "Right_Motor_OUT_A" I L 2050 5400 50
-F9 "Right_Motor_OUT_B" I L 2050 5500 50
-$EndSheet
-$Sheet
-S 5350 3700 1550 650
-U 6163ECBF
-F0 "GyroSensor" 50
-F1 "GyroSensor.sch" 50
-$EndSheet
+F2 "IR_Sensor_OUT1" I R 5800 2550 50
+F3 "IR_Sensor_OUT2" I R 5800 2650 50
+F4 "1.65V" I L 4400 2550 50
+F5 "IR_Sensor_IN1" O R 5800 2850 50
+F6 "IR_Sensor_IN2" O R 5800 2950 50
+F7 "IR_Sensor_IN3" O R 5800 3050 50
+F8 "IR_Sensor_IN4" O R 5800 3150 50
+$EndSheet
+Wire Wire Line
+	4150 2050 4150 2550
+Wire Wire Line
+	4150 2550 4400 2550
+Wire Wire Line
+	5800 2850 6000 2850
+Wire Wire Line
+	6000 2850 6000 2650
+Wire Wire Line
+	6000 2650 6450 2650
+Wire Wire Line
+	6450 2750 6050 2750
+Wire Wire Line
+	6050 2750 6050 2950
+Wire Wire Line
+	6050 2950 5800 2950
+Wire Wire Line
+	5800 3050 6100 3050
+Wire Wire Line
+	6100 3050 6100 2850
+Wire Wire Line
+	6100 2850 6450 2850
+Wire Wire Line
+	6450 2950 6150 2950
+Wire Wire Line
+	6150 2950 6150 3150
+Wire Wire Line
+	6150 3150 5800 3150
+Wire Wire Line
+	5800 3950 6450 3950
+Wire Wire Line
+	6450 4050 5800 4050
+Wire Wire Line
+	5800 4200 6450 4200
+Wire Wire Line
+	6450 4300 5800 4300
+Wire Wire Line
+	4100 4300 4050 4300
+Wire Wire Line
+	4050 4300 4050 4500
+Wire Wire Line
+	4050 4500 6450 4500
+Wire Wire Line
+	4100 4200 4000 4200
+Wire Wire Line
+	4000 4200 4000 4600
+Wire Wire Line
+	4000 4600 6450 4600
+Wire Wire Line
+	4050 3650 6450 3650
+Wire Wire Line
+	4000 3550 6450 3550
+Wire Wire Line
+	4000 3550 4000 4050
+Wire Wire Line
+	4000 4050 4100 4050
+Wire Wire Line
+	4100 3950 4050 3950
+Wire Wire Line
+	4050 3950 4050 3650
+$Sheet
+S 6450 1400 1400 3250
+U 61651214
+F0 "MicroController" 50
+F1 "MicroController.sch" 50
+F2 "LED1" O R 7850 1650 50
+F3 "LED2" O R 7850 1750 50
+F4 "LED3" O R 7850 1850 50
+F5 "LED4" O R 7850 1950 50
+F6 "LED5" O R 7850 2050 50
+F7 "LED6" O R 7850 2150 50
+F8 "IMU_CLK" O R 7850 3850 50
+F9 "IMU_MOSI" O R 7850 4000 50
+F10 "IMU_MISO" O R 7850 4250 50
+F11 "IMU_CS" O R 7850 4400 50
+F12 "UART_TX" O R 7850 2650 50
+F13 "UART_RX" I R 7850 2750 50
+F14 "SWCLK" O R 7850 2950 50
+F15 "SWDIO" O R 7850 3050 50
+F16 "NRST" I R 7850 3150 50
+F17 "BAT_REF" I L 6450 1650 50
+F18 "IR_Sensor_IN1" I L 6450 2650 50
+F19 "IR_Sensor_IN2" I L 6450 2750 50
+F20 "IR_Sensor_IN3" I L 6450 2850 50
+F21 "IR_Sensor_IN4" I L 6450 2950 50
+F22 "Left_EncoderA" I L 6450 3950 50
+F23 "Left_EncoderB" I L 6450 4050 50
+F24 "Right_EncoderA" I L 6450 4200 50
+F25 "Right_EncoderB" I L 6450 4300 50
+F26 "Right_Motor_OUT1" I L 6450 4600 50
+F27 "Right_Motor_OUT2" I L 6450 4500 50
+F28 "Left_Motor_OUT1" I L 6450 3650 50
+F29 "Left_Motor_OUT2" I L 6450 3550 50
+F30 "Buzzer" O R 7850 1500 50
+F31 "IR_Sensor_OUT1" O L 6450 2150 50
+F32 "IR_Sensor_OUT2" O L 6450 2250 50
+$EndSheet
+Wire Wire Line
+	7850 1500 9000 1500
+Wire Wire Line
+	5950 2650 5950 2250
+Wire Wire Line
+	5950 2250 6450 2250
+Wire Wire Line
+	5800 2650 5950 2650
+Wire Wire Line
+	6450 2150 5900 2150
+Wire Wire Line
+	5900 2150 5900 2550
+Wire Wire Line
+	5900 2550 5800 2550
 $EndSCHEMATC

Commit message: Make netlist
Changed lines of the file:
@@
 $EndSheet
 $Sheet
-S 9000 2450 550  800
+S 9000 2550 550  800
 U 6169318F
 F0 "Communication" 50
 F1 "Communication.sch" 50
-F2 "UART_TX" I L 9000 2650 50
-F3 "UART_RX" O L 9000 2750 50
-F4 "SWCLK" I L 9000 2950 50
-F5 "SWDIO" B L 9000 3050 50
-F6 "NRST" O L 9000 3150 50
+F2 "UART_TX" I L 9000 2750 50
+F3 "UART_RX" O L 9000 2850 50
+F4 "SWCLK" I L 9000 3050 50
+F5 "SWDIO" B L 9000 3150 50
+F6 "NRST" O L 9000 3250 50
 $EndSheet
 Wire Wire Line
@@
 	7850 1650 9000 1650
 $Sheet
-S 9000 1400 550  850
+S 9000 1400 550  1000
 U 61682BF7
 F0 "Debug" 50
@@
 F7 "Buzzer" I L 9000 1500 50
 F8 "LED6" I L 9000 2150 50
+F9 "Button1" O L 9000 2250 50
+F10 "Button2" O L 9000 2350 50
 $EndSheet
 Wire Wire Line
@@
 $EndSheet
 Wire Wire Line
-	9000 2750 7850 2750
-Wire Wire Line
-	7850 2650 9000 2650
-Wire Wire Line
 	7850 3850 8100 3850
 Wire Wire Line
@@
 Wire Wire Line
 	7850 4400 8100 4400
-Wire Wire Line
-	7850 2950 9000 2950
-Wire Wire Line
-	7850 3150 9000 3150
-Wire Wire Line
-	9000 3050 7850 3050
 Wire Wire Line
 	5800 1650 6450 1650
@@
 F8 "IMU_CLK" O R 7850 3850 50
 F9 "IMU_MOSI" O R 7850 4000 50
-F10 "IMU_MISO" O R 7850 4250 50
+F10 "IMU_MISO" I R 7850 4250 50
 F11 "IMU_CS" O R 7850 4400 50
-F12 "UART_TX" O R 7850 2650 50
-F13 "UART_RX" I R 7850 2750 50
-F14 "SWCLK" O R 7850 2950 50
-F15 "SWDIO" O R 7850 3050 50
-F16 "NRST" I R 7850 3150 50
+F12 "UART_TX" O R 7850 2750 50
+F13 "UART_RX" I R 7850 2850 50
+F14 "SWCLK" O R 7850 3050 50
+F15 "SWDIO" B R 7850 3150 50
+F16 "NRST" I R 7850 3250 50
 F17 "BAT_REF" I L 6450 1650 50
 F18 "IR_Sensor_IN1" I L 6450 2650 50
@@
 F24 "Right_EncoderA" I L 6450 4200 50
 F25 "Right_EncoderB" I L 6450 4300 50
-F26 "Right_Motor_OUT1" I L 6450 4600 50
-F27 "Right_Motor_OUT2" I L 6450 4500 50
-F28 "Left_Motor_OUT1" I L 6450 3650 50
-F29 "Left_Motor_OUT2" I L 6450 3550 50
+F26 "Right_Motor_OUT1" O L 6450 4600 50
+F27 "Right_Motor_OUT2" O L 6450 4500 50
+F28 "Left_Motor_OUT1" O L 6450 3650 50
+F29 "Left_Motor_OUT2" O L 6450 3550 50
 F30 "Buzzer" O R 7850 1500 50
 F31 "IR_Sensor_OUT1" O L 6450 2150 50
 F32 "IR_Sensor_OUT2" O L 6450 2250 50
+F33 "Button1" I R 7850 2250 50
+F34 "Button2" I R 7850 2350 50
 $EndSheet
 Wire Wire Line
@@
 Wire Wire Line
 	5900 2550 5800 2550
+Wire Wire Line
+	7850 2750 9000 2750
+Wire Wire Line
+	7850 2850 9000 2850
+Wire Wire Line
+	7850 3050 9000 3050
+Wire Wire Line
+	7850 3150 9000 3150
+Wire Wire Line
+	7850 3250 9000 3250
+Wire Wire Line
+	7850 2250 9000 2250
+Wire Wire Line
+	9000 2350 7850 2350
 $EndSCHEMATC
