File: pcb/ZeroPCB.kicad_pcb (KiCad board)
At the start: 2 copper layers, 84 x 100 mm, 92 parts, among them J1 BATTERY1, J10 UART, J11 ST_LINK, J12 DRV8835_Left, J13 DRV8835_Right, J2 BATTERY2, J3 VX07803-500, J4 Left_Motor, J5 Right_Motor, J6 GyroLeft, J7 GyroRight, J8 CN2_Right, J9 CN1_Left, Q1 IRLML6402, Q2 IRFML8244, Q3 IRFML8244, Q4 IRFML8244, SW1 POWER_SWITCH, SW2 Button1, SW3 Button2, U1 NJU77701F, U2 NJM2746, U3 NJU7098, U4 NJU7098, U5 NJU7098, U6 NJU7098

Commit message: Update schematic
Parts:
- removed J12: DRV8835_Left, Pin_Headers:Pin_Header_Straight_1x06_Pitch2.54mm
- removed J13: DRV8835_Right, Pin_Headers:Pin_Header_Straight_1x06_Pitch2.54mm
- removed J9: CN1_Left, Pin_Headers:Pin_Header_Straight_2x13_Pitch2.54mm
- J6: value GyroLeft -> L3GD20H; footprint Pin_Headers:Pin_Header_Straight_1x04_Pitch2.54mm -> Zero_Module:L3GD20HBoard
- J7: value GyroRight -> STM32F405Board; footprint Pin_Headers:Pin_Header_Straight_1x04_Pitch2.54mm -> Zero_Module:STM32F405Board
- J8: value CN2_Right -> DRV8835; footprint Pin_Headers:Pin_Header_Straight_2x13_Pitch2.54mm -> Zero_Module:DRV8835Board
- moved J8 51.7 mm to (88.6, 114.7)
- moved J7 44.9 mm to (87.4, 88.6), turned to 90 degrees
- moved J6 4.10 mm to (96.3, 44.1)
Connections:
- J4 pad 1: Net-(J12-Pad3) -> Net-(J4-Pad1)
- J4 pad 2: Net-(J12-Pad2) -> Net-(J4-Pad2)
- J5 pad 1: Net-(J12-Pad5) -> Net-(J5-Pad1)
- J5 pad 2: Net-(J12-Pad4) -> Net-(J5-Pad2)
- J7 pad 2: (no net) -> +3V3
- J7 pad 3: (no net) -> /IRSensor/IR_Sensor_IN1
- J7 pad 4: /GyroSensor/IMU_CS -> /IRSensor/IR_Sensor_IN2
- J8 pad 1: GND -> +BATT
- J8 pad 10: /GyroSensor/IMU_MOSI -> /MicroController/Left_Motor_OUT1
- J8 pad 11: (no net) -> GND
- J8 pad 12: (no net) -> +3V3
- J8 pad 2: +3V3 -> Net-(J4-Pad2)
- J8 pad 3: /MicroController/Left_EncoderA -> Net-(J4-Pad1)
- J8 pad 4: /MicroController/Left_EncoderB -> Net-(J5-Pad2)
- J8 pad 5: /IRSensor/IR_Sensor_OUT1 -> Net-(J5-Pad1)
- J8 pad 6: /IRSensor/IR_Sensor_OUT2 -> GND
- J8 pad 7: /GyroSensor/IMU_CS -> /MicroController/Right_Motor_OUT2
- J8 pad 8: /GyroSensor/IMU_CLK -> /MicroController/Right_Motor_OUT1
- J8 pad 9: /GyroSensor/IMU_MISO -> /MicroController/Left_Motor_OUT2

Commit message: Update
Parts:
- C13: footprint Capacitors_SMD:C_0603_HandSoldering -> Capacitors_SMD:C_0805_HandSoldering
- D16: value LED4 -> ButtonLED1
- D17: value LED4 -> ButtonLED2
- moved J11 172.6 mm to (104.5, 120.0), turned to 90 degrees
- moved J10 164.0 mm to (104.5, 69.3), turned to 90 degrees
- moved Q1 141.3 mm to (108.0, 110.0)
- moved R5 140.7 mm to (111.5, 98.3), turned to 270 degrees
- moved R1 140.6 mm to (104.2, 110.0), turned to 90 degrees
- moved U1 140.0 mm to (106.7, 93.9), turned to 90 degrees
- moved R19 137.4 mm to (154.8, 128.0)
- moved C6 132.4 mm to (154.7, 123.5), turned to 180 degrees
- moved J1 131.8 mm to (109.7, 115.0), turned to 270 degrees
- moved J2 129.8 mm to (109.7, 123.3), turned to 270 degrees
- moved C2 128.8 mm to (107.0, 99.5), turned to 180 degrees
- moved R4 128.6 mm to (111.5, 93.3), turned to 270 degrees
- moved U4 128.3 mm to (155.0, 131.5)
- moved R16 126.6 mm to (150.7, 63.5), turned to 270 degrees
- moved R26 123.8 mm to (100.0, 72.4), turned to 90 degrees
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Other:
- board size 84 x 100 mm -> 100 x 84 mm

Commit message: Run autorouter
Parts:
- moved R21 2.50 mm to (181.7, 119.5)
- moved C9 2.50 mm to (181.7, 124.0)
- moved L1 2.43 mm to (144.0, 103.5)
- moved J3 2.24 mm to (144.0, 91.8)
- moved C13 1.26 mm to (144.1, 85.2)
- moved R15 1.25 mm to (168.8, 107.0)
- moved R12 1.25 mm to (168.7, 88.5)
- moved R13 1.25 mm to (168.7, 100.5)
- moved Q2 1.23 mm to (168.8, 85.0)
- moved C12 1.23 mm to (144.0, 88.3)
- moved Q3 1.23 mm to (168.8, 103.8)
- moved C8 1.04 mm to (181.5, 65.5)
- moved J2 1.00 mm to (110.7, 123.2)
- moved J1 1.00 mm to (110.7, 115.0)
- moved R14 0.98 mm to (168.8, 81.5)
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Routing:
- net GND: track 0.00 -> 530.1 mm, vias 0 -> 15
- net +3V3: track 0.00 -> 285.2 mm, vias 0 -> 2
- net /IRSensor/1.65V: track 0.00 -> 195.9 mm, vias 0 -> 2
- net +3.3VA: track 0.00 -> 168.4 mm, vias 0 -> 1
- net /Communication/SWDIO: track 0.00 -> 167.4 mm, vias 0 -> 3
- net +BATT: track 0.00 -> 143.3 mm
- net /Communication/SWCLK: track 0.00 -> 139.5 mm, vias 0 -> 3
- net /MicroController/Left_EncoderA: track 0.00 -> 107.8 mm, vias 0 -> 1
- net /Debug/LED2: track 0.00 -> 94.3 mm, vias 0 -> 1
- net /Debug/Button1: track 0.00 -> 89.8 mm, vias 0 -> 1
- net /MicroController/Left_Motor_OUT1: track 0.00 -> 88.9 mm, vias 0 -> 1
- net /MicroController/Left_Motor_OUT2: track 0.00 -> 88.8 mm, vias 0 -> 1
- net /Debug/LED1: track 0.00 -> 87.0 mm, vias 0 -> 1
- net /Debug/LED3: track 0.00 -> 83.8 mm, vias 0 -> 1
- net /MicroController/Left_EncoderB: track 0.00 -> 77.1 mm, vias 0 -> 2
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- added copper zone on B.Cu, net GND
- added copper zone on F.Cu, net GND
Other:
- outline, holes or cut-outs redrawn
- net class Power added: clearance 0.2, trace_width 0.4, via_dia 0.8, via_drill 0.4

Commit message: Update pcb
Parts:
- added C14: 0.1u, Capacitors_SMD:C_0603_HandSoldering, F.Cu at (110.0, 104.8)
- added C15: 0.1u, Capacitors_SMD:C_0603_HandSoldering, F.Cu at (156.8, 83.5)
- added C16: 10u, Capacitors_SMD:C_0603_HandSoldering, F.Cu at (110.0, 106.8)
- added C17: 10u, Capacitors_SMD:C_0603_HandSoldering, F.Cu at (156.8, 81.5)
- added C18: 2.2u, Capacitors_SMD:C_0603_HandSoldering, F.Cu at (135.4, 103.7)
- added J12: GND_PIN, Pin_Headers:Pin_Header_Straight_1x01_Pitch2.54mm, F.Cu at (100.7, 103.6)
- added J9: BATT_PIN, Pin_Headers:Pin_Header_Straight_1x01_Pitch2.54mm, F.Cu at (100.6, 85.8)
- LS1: value Speaker -> SMT-0440
- moved U6 0.51 mm to (177.2, 120.0)
Connections:
- D6 pad 1: Net-(C4-Pad2) -> +3.3VA
- D6 pad 2: +3.3VA -> Net-(C4-Pad2)
- D7 pad 1: Net-(C6-Pad2) -> +3.3VA
- D7 pad 2: +3.3VA -> Net-(C6-Pad2)
- D8 pad 1: Net-(C8-Pad2) -> +3.3VA
- D8 pad 2: +3.3VA -> Net-(C8-Pad2)
- D9 pad 1: Net-(C9-Pad2) -> +3.3VA
- D9 pad 2: +3.3VA -> Net-(C9-Pad2)
- J7 pad 25: (no net) -> +3V3
Routing:
- net +3V3: track 285.2 -> 323.5 mm, vias 2 -> 3
- net Net-(J1-Pad1): track 8.37 -> 35.5 mm, vias 0 -> 1
- net +3.3VA: track 168.4 -> 184.3 mm
- net GND: track 530.1 -> 515.1 mm, vias 15 -> 37
- net Net-(C9-Pad2): track 29.9 -> 23.6 mm
- net Net-(C11-Pad2): track 9.22 -> 7.30 mm
- net Net-(C6-Pad2): track 15.3 -> 13.9 mm
- net Net-(C8-Pad2): track 22.7 -> 21.9 mm
- net /Debug/LED4: track 60.8 -> 61.5 mm
- net /IRSensor/1.65V: track 195.9 -> 195.3 mm
- net /IRSensor/IR_Sensor_IN4: track 75.3 -> 74.7 mm
Other:
- board text added: "2021-10-31 Dangoromouse Zero aka Cheese Tutorial Mouse"

Commit message: Update
Parts:
- added G***: LOGO, Zero_Module:cheese_logo_regular, B.Cu at (134.4, 94.2)
