File: pcb/Communication.sch (KiCad schematic (older format))
At the start: 2 parts, among them J10 UART, J11 ST_LINK

Commit message: Make netlist
Parts:
- J10, J11: footprint (none) -> Connector_JST:JST_SH_BM04B-SRSS-TB_1x04-1MP_P1.00mm_Vertical
Changed lines of the file:
@@
 $Descr A4 11693 8268
 encoding utf-8
-Sheet 5 8
+Sheet 4 8
 Title ""
 Date ""
@@
 F 0 "J10" H 3328 2126 50  0000 L CNN
 F 1 "UART" H 3328 2035 50  0000 L CNN
-F 2 "" H 3300 2150 50  0001 C CNN
+F 2 "Connector_JST:JST_SH_BM04B-SRSS-TB_1x04-1MP_P1.00mm_Vertical" H 3300 2150 50  0001 C CNN
 F 3 "~" H 3300 2150 50  0001 C CNN
 	1    3300 2150
@@
 F 0 "J11" H 3328 2726 50  0000 L CNN
 F 1 "ST_LINK" H 3328 2635 50  0000 L CNN
-F 2 "" H 3300 2750 50  0001 C CNN
+F 2 "Connector_JST:JST_SH_BM04B-SRSS-TB_1x04-1MP_P1.00mm_Vertical" H 3300 2750 50  0001 C CNN
 F 3 "~" H 3300 2750 50  0001 C CNN
 	1    3300 2750

Commit message: Write about where to buy the parts
Parts:
- J10, J11: Buy (none) -> https://www.sengoku.co.jp/mod/sgk_cart/detail.php?code=EEHD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; Vendor (none) -> https://www.sengoku.co.jp/mod/sgk_cart/detail.php?code=EEHD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
Changed lines of the file:
@@
 F 1 "UART" H 3328 2035 50  0000 L CNN
 F 2 "Connector_JST:JST_SH_BM04B-SRSS-TB_1x04-1MP_P1.00mm_Vertical" H 3300 2150 50  0001 C CNN
-F 3 "~" H 3300 2150 50  0001 C CNN
+F 3 "https://www.sengoku.co.jp/mod/sgk_cart/detail.php?code=EEHD-0KNJ" H 3300 2150 50  0001 C CNN
+F 4 "https://www.sengoku.co.jp/mod/sgk_cart/detail.php?code=EEHD-0KNJ" H 3300 2150 50  0001 C CNN "Buy"
+F 5 "https://www.sengoku.co.jp/mod/sgk_cart/detail.php?code=EEHD-0KNJ" H 3300 2150 50  0001 C CNN "Vendor"
 	1    3300 2150
 	1    0    0    -1
@@
 F 1 "ST_LINK" H 3328 2635 50  0000 L CNN
 F 2 "Connector_JST:JST_SH_BM04B-SRSS-TB_1x04-1MP_P1.00mm_Vertical" H 3300 2750 50  0001 C CNN
-F 3 "~" H 3300 2750 50  0001 C CNN
+F 3 "https://www.sengoku.co.jp/mod/sgk_cart/detail.php?code=EEHD-0KNJ" H 3300 2750 50  0001 C CNN
+F 4 "https://www.sengoku.co.jp/mod/sgk_cart/detail.php?code=EEHD-0KNJ" H 3300 2750 50  0001 C CNN "Buy"
+F 5 "https://www.sengoku.co.jp/mod/sgk_cart/detail.php?code=EEHD-0KNJ" H 3300 2750 50  0001 C CNN "Vendor"
 	1    3300 2750
 	1    0    0    -1
