File: pcb/Debug.sch (KiCad schematic (older format))
At the start: 15 parts, among them Q4 IRFML8244

Commit message: Make netlist
Parts:
- added D16, D17: LED4, LEDs:LED_0603_HandSoldering, symbol Device:LED
- added R31, R33: 1k, Resistors_SMD:R_0603_HandSoldering, symbol Device:R
- added R32, R34: 10k, Resistors_SMD:R_0603_HandSoldering, symbol Device:R
- added SW2: Button1, Buttons_Switches_SMD:SW_SPST_EVQP2, symbol REF1933:SW_Push
- added SW3: Button2, Buttons_Switches_SMD:SW_SPST_EVQP2, symbol REF1933:SW_Push
- D10: value LED -> LED1; footprint (none) -> LEDs:LED_0603_HandSoldering
- D11: value LED -> LED2; footprint (none) -> LEDs:LED_0603_HandSoldering
- D12: value LED -> LED3; footprint (none) -> LEDs:LED_0603_HandSoldering
- D13: value LED -> LED4; footprint (none) -> LEDs:LED_0603_HandSoldering
- D14: value LED -> LED5; footprint (none) -> LEDs:LED_0603_HandSoldering
- D15: value LED -> LED6; footprint (none) -> LEDs:LED_0603_HandSoldering
- LS1: footprint (none) -> PUI_Audio:SMT-0440-S-R
- Q4: footprint (none) -> TO_SOT_Packages_SMD:SOT-23
- R24, R25, R26, R27, R28, R29, R30: footprint (none) -> Resistors_SMD:R_0603_HandSoldering
Connections:
- net +3V3: now also SW2.1, SW3.1
- net GND: now also D16.1 (K), D17.1 (K), R32.1, R34.1
- new net: D16.2 (A), R31.1
- new net: D17.2 (A), R33.1
- new net Button1: R31.2, R32.2, SW2.2
- new net Button2: R33.2, R34.2, SW3.2
Changed lines of the file:
@@
 P 3150 2550
 F 0 "D10" H 3143 2295 50  0000 C CNN
-F 1 "LED" H 3143 2386 50  0000 C CNN
-F 2 "" H 3150 2550 50  0001 C CNN
+F 1 "LED1" H 3143 2386 50  0000 C CNN
+F 2 "LEDs:LED_0603_HandSoldering" H 3150 2550 50  0001 C CNN
 F 3 "~" H 3150 2550 50  0001 C CNN
 	1    3150 2550
@@
 F 0 "R24" V 2643 2550 50  0000 C CNN
 F 1 "1k" V 2850 2550 50  0000 C CNN
-F 2 "" V 2780 2550 50  0001 C CNN
+F 2 "Resistors_SMD:R_0603_HandSoldering" V 2780 2550 50  0001 C CNN
 F 3 "~" H 2850 2550 50  0001 C CNN
 	1    2850 2550
@@
 P 3150 2900
 F 0 "D11" H 3143 2645 50  0000 C CNN
-F 1 "LED" H 3143 2736 50  0000 C CNN
-F 2 "" H 3150 2900 50  0001 C CNN
+F 1 "LED2" H 3143 2736 50  0000 C CNN
+F 2 "LEDs:LED_0603_HandSoldering" H 3150 2900 50  0001 C CNN
 F 3 "~" H 3150 2900 50  0001 C CNN
 	1    3150 2900
@@
 F 0 "R25" V 2643 2900 50  0000 C CNN
 F 1 "1k" V 2850 2900 50  0000 C CNN
-F 2 "" V 2780 2900 50  0001 C CNN
+F 2 "Resistors_SMD:R_0603_HandSoldering" V 2780 2900 50  0001 C CNN
 F 3 "~" H 2850 2900 50  0001 C CNN
 	1    2850 2900
@@
 P 3150 3250
 F 0 "D12" H 3143 2995 50  0000 C CNN
-F 1 "LED" H 3143 3086 50  0000 C CNN
-F 2 "" H 3150 3250 50  0001 C CNN
+F 1 "LED3" H 3143 3086 50  0000 C CNN
+F 2 "LEDs:LED_0603_HandSoldering" H 3150 3250 50  0001 C CNN
 F 3 "~" H 3150 3250 50  0001 C CNN
 	1    3150 3250
@@
 F 0 "R26" V 2643 3250 50  0000 C CNN
 F 1 "1k" V 2850 3250 50  0000 C CNN
-F 2 "" V 2780 3250 50  0001 C CNN
+F 2 "Resistors_SMD:R_0603_HandSoldering" V 2780 3250 50  0001 C CNN
 F 3 "~" H 2850 3250 50  0001 C CNN
 	1    2850 3250
@@
 P 3150 3600
 F 0 "D13" H 3143 3345 50  0000 C CNN
-F 1 "LED" H 3143 3436 50  0000 C CNN
-F 2 "" H 3150 3600 50  0001 C CNN
+F 1 "LED4" H 3143 3436 50  0000 C CNN
+F 2 "LEDs:LED_0603_HandSoldering" H 3150 3600 50  0001 C CNN
 F 3 "~" H 3150 3600 50  0001 C CNN
 	1    3150 3600
@@
 F 0 "R27" V 2643 3600 50  0000 C CNN
 F 1 "1k" V 2850 3600 50  0000 C CNN
-F 2 "" V 2780 3600 50  0001 C CNN
+F 2 "Resistors_SMD:R_0603_HandSoldering" V 2780 3600 50  0001 C CNN
 F 3 "~" H 2850 3600 50  0001 C CNN
 	1    2850 3600
@@
 P 3150 3950
 F 0 "D14" H 3143 3695 50  0000 C CNN
-F 1 "LED" H 3143 3786 50  0000 C CNN
-F 2 "" H 3150 3950 50  0001 C CNN
+F 1 "LED5" H 3143 3786 50  0000 C CNN
+F 2 "LEDs:LED_0603_HandSoldering" H 3150 3950 50  0001 C CNN
 F 3 "~" H 3150 3950 50  0001 C CNN
 	1    3150 3950
@@
 F 0 "R28" V 2643 3950 50  0000 C CNN
 F 1 "1k" V 2850 3950 50  0000 C CNN
-F 2 "" V 2780 3950 50  0001 C CNN
+F 2 "Resistors_SMD:R_0603_HandSoldering" V 2780 3950 50  0001 C CNN
 F 3 "~" H 2850 3950 50  0001 C CNN
 	1    2850 3950
@@
 F 0 "LS1" H 4920 2446 50  0000 L CNN
 F 1 "Speaker" H 4920 2355 50  0000 L CNN
-F 2 "" H 4750 2250 50  0001 C CNN
+F 2 "PUI_Audio:SMT-0440-S-R" H 4750 2250 50  0001 C CNN
 F 3 "~" H 4740 2400 50  0001 C CNN
 	1    4750 2450
@@
 F 0 "Q4" H 4641 3296 50  0000 L CNN
 F 1 "IRFML8244" H 4641 3205 50  0000 L CNN
-F 2 "" H 4650 3350 50  0001 C CNN
+F 2 "TO_SOT_Packages_SMD:SOT-23" H 4650 3350 50  0001 C CNN
 F 3 "~" H 4450 3250 50  0001 C CNN
 	1    4450 3250
@@
 F 0 "R29" H 4620 2946 50  0000 L CNN
 F 1 "1k" H 4620 2855 50  0000 L CNN
-F 2 "" V 4480 2900 50  0001 C CNN
+F 2 "Resistors_SMD:R_0603_HandSoldering" V 4480 2900 50  0001 C CNN
 F 3 "~" H 4550 2900 50  0001 C CNN
 	1    4550 2900
@@
 LED5
 $Comp
-L Device:LED D15
-U 1 1 616C844D
-P 3150 4350
-F 0 "D15" H 3143 4095 50  0000 C CNN
-F 1 "LED" H 3143 4186 50  0000 C CNN
-F 2 "" H 3150 4350 50  0001 C CNN
-F 3 "~" H 3150 4350 50  0001 C CNN
-	1    3150 4350
-	-1   0    0    1
-$EndComp
-$Comp
 L Device:R R30
 U 1 1 616C8453
@@
 F 0 "R30" V 2643 4350 50  0000 C CNN
 F 1 "1k" V 2850 4350 50  0000 C CNN
-F 2 "" V 2780 4350 50  0001 C CNN
+F 2 "Resistors_SMD:R_0603_HandSoldering" V 2780 4350 50  0001 C CNN
 F 3 "~" H 2850 4350 50  0001 C CNN
 	1    2850 4350
@@
 Text HLabel 2700 4350 0    50   Input ~ 0
 LED6
+$Comp
+L Device:LED D15
+U 1 1 616C844D
+P 3150 4350
+F 0 "D15" H 3143 4095 50  0000 C CNN
+F 1 "LED6" H 3143 4186 50  0000 C CNN
+F 2 "LEDs:LED_0603_HandSoldering" H 3150 4350 50  0001 C CNN
+F 3 "~" H 3150 4350 50  0001 C CNN
+	1    3150 4350
+	-1   0    0    1
+$EndComp
+$Comp
+L REF1933:SW_Push SW2
+U 1 1 61800D4F
+P 6750 3300
+F 0 "SW2" V 6704 3448 50  0000 L CNN
+F 1 "Button1" V 6795 3448 50  0000 L CNN
+F 2 "Buttons_Switches_SMD:SW_SPST_EVQP2" H 6750 3500 50  0001 C CNN
+F 3 "" H 6750 3500 50  0001 C CNN
+	1    6750 3300
+	0    1    1    0
+$EndComp
+$Comp
+L Device:LED D16
+U 1 1 61805D2D
+P 6350 3950
+F 0 "D16" H 6343 3695 50  0000 C CNN
+F 1 "LED4" H 6343 3786 50  0000 C CNN
+F 2 "LEDs:LED_0603_HandSoldering" H 6350 3950 50  0001 C CNN
+F 3 "~" H 6350 3950 50  0001 C CNN
+	1    6350 3950
+	0    -1   -1   0
+$EndComp
+$Comp
+L Device:R R31
+U 1 1 61805D33
+P 6350 3650
+F 0 "R31" V 6143 3650 50  0000 C CNN
+F 1 "1k" V 6350 3650 50  0000 C CNN
+F 2 "Resistors_SMD:R_0603_HandSoldering" V 6280 3650 50  0001 C CNN
+F 3 "~" H 6350 3650 50  0001 C CNN
+	1    6350 3650
+	-1   0    0    1
+$EndComp
+Wire Wire Line
+	6350 3500 6750 3500
+$Comp
+L Device:R R32
+U 1 1 6180DD4C
+P 6750 3950
+F 0 "R32" V 6543 3950 50  0000 C CNN
+F 1 "10k" V 6750 3950 50  0000 C CNN
+F 2 "Resistors_SMD:R_0603_HandSoldering" V 6680 3950 50  0001 C CNN
+F 3 "~" H 6750 3950 50  0001 C CNN
+	1    6750 3950
+	-1   0    0    1
+$EndComp
+Wire Wire Line
+	6750 3500 6750 3800
+Connection ~ 6750 3500
+Wire Wire Line
+	6750 4100 6350 4100
+$Comp
+L power:GND #PWR050
+U 1 1 61810E8B
+P 6350 4100
+F 0 "#PWR050" H 6350 3850 50  0001 C CNN
+F 1 "GND" H 6355 3927 50  0000 C CNN
+F 2 "" H 6350 4100 50  0001 C CNN
+F 3 "" H 6350 4100 50  0001 C CNN
+	1    6350 4100
+	1    0    0    -1
+$EndComp
+Connection ~ 6350 4100
+$Comp
+L power:+3.3V #PWR051
+U 1 1 61811563
+P 6750 3100
+F 0 "#PWR051" H 6750 2950 50  0001 C CNN
+F 1 "+3.3V" H 6765 3273 50  0000 C CNN
+F 2 "" H 6750 3100 50  0001 C CNN
+F 3 "" H 6750 3100 50  0001 C CNN
+	1    6750 3100
+	1    0    0    -1
+$EndComp
+Text HLabel 6750 3500 2    50   Output ~ 0
+Button1
+$Comp
+L REF1933:SW_Push SW3
+U 1 1 6181A7BA
+P 7700 3300
+F 0 "SW3" V 7654 3448 50  0000 L CNN
+F 1 "Button2" V 7745 3448 50  0000 L CNN
+F 2 "Buttons_Switches_SMD:SW_SPST_EVQP2" H 7700 3500 50  0001 C CNN
+F 3 "" H 7700 3500 50  0001 C CNN
+	1    7700 3300
+	0    1    1    0
+$EndComp
+$Comp
+L Device:LED D17
+U 1 1 6181A7C0
+P 7300 3950
+F 0 "D17" H 7293 3695 50  0000 C CNN
+F 1 "LED4" H 7293 3786 50  0000 C CNN
+F 2 "LEDs:LED_0603_HandSoldering" H 7300 3950 50  0001 C CNN
+F 3 "~" H 7300 3950 50  0001 C CNN
+	1    7300 3950
+	0    -1   -1   0
+$EndComp
+$Comp
+L Device:R R33
+U 1 1 6181A7C6
+P 7300 3650
+F 0 "R33" V 7093 3650 50  0000 C CNN
+F 1 "1k" V 7300 3650 50  0000 C CNN
+F 2 "Resistors_SMD:R_0603_HandSoldering" V 7230 3650 50  0001 C CNN
+F 3 "~" H 7300 3650 50  0001 C CNN
+	1    7300 3650
+	-1   0    0    1
+$EndComp
+Wire Wire Line
+	7300 3500 7700 3500
+$Comp
+L Device:R R34
+U 1 1 6181A7CD
+P 7700 3950
+F 0 "R34" V 7493 3950 50  0000 C CNN
+F 1 "10k" V 7700 3950 50  0000 C CNN
+F 2 "Resistors_SMD:R_0603_HandSoldering" V 7630 3950 50  0001 C CNN
+F 3 "~" H 7700 3950 50  0001 C CNN
+	1    7700 3950
+	-1   0    0    1
+$EndComp
+Wire Wire Line
+	7700 3500 7700 3800
+Connection ~ 7700 3500
+Wire Wire Line
+	7700 4100 7300 4100
+$Comp
+L power:GND #PWR052
+U 1 1 6181A7D6
+P 7300 4100
+F 0 "#PWR052" H 7300 3850 50  0001 C CNN
+F 1 "GND" H 7305 3927 50  0000 C CNN
+F 2 "" H 7300 4100 50  0001 C CNN
+F 3 "" H 7300 4100 50  0001 C CNN
+	1    7300 4100
+	1    0    0    -1
+$EndComp
+Connection ~ 7300 4100
+$Comp
+L power:+3.3V #PWR053
+U 1 1 6181A7DD
+P 7700 3100
+F 0 "#PWR053" H 7700 2950 50  0001 C CNN
+F 1 "+3.3V" H 7715 3273 50  0000 C CNN
+F 2 "" H 7700 3100 50  0001 C CNN
+F 3 "" H 7700 3100 50  0001 C CNN
+	1    7700 3100
+	1    0    0    -1
+$EndComp
+Text HLabel 7700 3500 2    50   Output ~ 0
+Button2
 $EndSCHEMATC

Commit message: Update
Parts:
- D16: value LED4 -> ButtonLED1
- D17: value LED4 -> ButtonLED2
Changed lines of the file:
@@
 P 6350 3950
 F 0 "D16" H 6343 3695 50  0000 C CNN
-F 1 "LED4" H 6343 3786 50  0000 C CNN
+F 1 "ButtonLED1" H 6343 3786 50  0000 C CNN
 F 2 "LEDs:LED_0603_HandSoldering" H 6350 3950 50  0001 C CNN
 F 3 "~" H 6350 3950 50  0001 C CNN
@@
 P 7300 3950
 F 0 "D17" H 7293 3695 50  0000 C CNN
-F 1 "LED4" H 7293 3786 50  0000 C CNN
+F 1 "ButtonLED2" H 7293 3786 50  0000 C CNN
 F 2 "LEDs:LED_0603_HandSoldering" H 7300 3950 50  0001 C CNN
 F 3 "~" H 7300 3950 50  0001 C CNN

Commit message: Update pcb
Parts:
- LS1: value Speaker -> SMT-0440
Changed lines of the file:
@@
 P 4750 2450
 F 0 "LS1" H 4920 2446 50  0000 L CNN
-F 1 "Speaker" H 4920 2355 50  0000 L CNN
+F 1 "SMT-0440" H 4920 2355 50  0000 L CNN
 F 2 "PUI_Audio:SMT-0440-S-R" H 4750 2250 50  0001 C CNN
 F 3 "~" H 4740 2400 50  0001 C CNN

Commit message: Write about where to buy the parts
Parts:
- D10, D11, D12, D13, D14, D15, D16, D17: Buy (none) -> https://akizukidenshi.com/catalog/g/gI-11879/; Vendor (none) -> https://akizukidenshi.com/catalog/g/gI-11879/
- LS1: Buy (none) -> https://www.digikey.jp/ja/products/detail/pui-audio-inc/SMT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; Vendor (none) -> https://www.digikey.jp/ja/products/detail/pui-audio-inc/SMT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
- Q4: Buy (none) -> https://akizukidenshi.com/catalog/g/gI-06051/; Vendor (none) -> https://akizukidenshi.com/catalog/g/gI-06051/
- R24, R25, R26, R27, R28, R29, R30, R31, R33: Buy (none) -> https://akizukidenshi.com/catalog/g/gR-14122/; Vendor (none) -> https://akizukidenshi.com/catalog/g/gR-14122/
- SW2, SW3: Buy (none) -> https://akizukidenshi.com/catalog/g/gP-06185/; Vendor (none) -> https://akizukidenshi.com/catalog/g/gP-06185/
Changed lines of the file:
@@
 F 1 "LED1" H 3143 2386 50  0000 C CNN
 F 2 "LEDs:LED_0603_HandSoldering" H 3150 2550 50  0001 C CNN
-F 3 "~" H 3150 2550 50  0001 C CNN
+F 3 "https://akizukidenshi.com/catalog/g/gI-11879/" H 3150 2550 50  0001 C CNN
+F 4 "https://akizukidenshi.com/catalog/g/gI-11879/" H 3150 2550 50  0001 C CNN "Buy"
+F 5 "https://akizukidenshi.com/catalog/g/gI-11879/" H 3150 2550 50  0001 C CNN "Vendor"
 	1    3150 2550
 	-1   0    0    1
@@
 F 1 "1k" V 2850 2550 50  0000 C CNN
 F 2 "Resistors_SMD:R_0603_HandSoldering" V 2780 2550 50  0001 C CNN
-F 3 "~" H 2850 2550 50  0001 C CNN
+F 3 "https://akizukidenshi.com/catalog/g/gR-14122/" H 2850 2550 50  0001 C CNN
+F 4 "https://akizukidenshi.com/catalog/g/gR-14122/" H 2850 2550 50  0001 C CNN "Buy"
+F 5 "https://akizukidenshi.com/catalog/g/gR-14122/" H 2850 2550 50  0001 C CNN "Vendor"
 	1    2850 2550
 	0    1    1    0
@@
 F 1 "LED2" H 3143 2736 50  0000 C CNN
 F 2 "LEDs:LED_0603_HandSoldering" H 3150 2900 50  0001 C CNN
-F 3 "~" H 3150 2900 50  0001 C CNN
+F 3 "https://akizukidenshi.com/catalog/g/gI-11879/" H 3150 2900 50  0001 C CNN
+F 4 "https://akizukidenshi.com/catalog/g/gI-11879/" H 3150 2900 50  0001 C CNN "Buy"
+F 5 "https://akizukidenshi.com/catalog/g/gI-11879/" H 3150 2900 50  0001 C CNN "Vendor"
 	1    3150 2900
 	-1   0    0    1
@@
 F 1 "1k" V 2850 2900 50  0000 C CNN
 F 2 "Resistors_SMD:R_0603_HandSoldering" V 2780 2900 50  0001 C CNN
-F 3 "~" H 2850 2900 50  0001 C CNN
+F 3 "https://akizukidenshi.com/catalog/g/gR-14122/" H 2850 2900 50  0001 C CNN
+F 4 "https://akizukidenshi.com/catalog/g/gR-14122/" H 2850 2900 50  0001 C CNN "Buy"
+F 5 "https://akizukidenshi.com/catalog/g/gR-14122/" H 2850 2900 50  0001 C CNN "Vendor"
 	1    2850 2900
 	0    1    1    0
@@
 F 1 "LED3" H 3143 3086 50  0000 C CNN
 F 2 "LEDs:LED_0603_HandSoldering" H 3150 3250 50  0001 C CNN
-F 3 "~" H 3150 3250 50  0001 C CNN
+F 3 "https://akizukidenshi.com/catalog/g/gI-11879/" H 3150 3250 50  0001 C CNN
+F 4 "https://akizukidenshi.com/catalog/g/gI-11879/" H 3150 3250 50  0001 C CNN "Buy"
+F 5 "https://akizukidenshi.com/catalog/g/gI-11879/" H 3150 3250 50  0001 C CNN "Vendor"
 	1    3150 3250
 	-1   0    0    1
@@
 F 1 "1k" V 2850 3250 50  0000 C CNN
 F 2 "Resistors_SMD:R_0603_HandSoldering" V 2780 3250 50  0001 C CNN
-F 3 "~" H 2850 3250 50  0001 C CNN
+F 3 "https://akizukidenshi.com/catalog/g/gR-14122/" H 2850 3250 50  0001 C CNN
+F 4 "https://akizukidenshi.com/catalog/g/gR-14122/" H 2850 3250 50  0001 C CNN "Buy"
+F 5 "https://akizukidenshi.com/catalog/g/gR-14122/" H 2850 3250 50  0001 C CNN "Vendor"
 	1    2850 3250
 	0    1    1    0
@@
 F 1 "LED4" H 3143 3436 50  0000 C CNN
 F 2 "LEDs:LED_0603_HandSoldering" H 3150 3600 50  0001 C CNN
-F 3 "~" H 3150 3600 50  0001 C CNN
+F 3 "https://akizukidenshi.com/catalog/g/gI-11879/" H 3150 3600 50  0001 C CNN
+F 4 "https://akizukidenshi.com/catalog/g/gI-11879/" H 3150 3600 50  0001 C CNN "Buy"
+F 5 "https://akizukidenshi.com/catalog/g/gI-11879/" H 3150 3600 50  0001 C CNN "Vendor"
 	1    3150 3600
 	-1   0    0    1
@@
 F 1 "1k" V 2850 3600 50  0000 C CNN
 F 2 "Resistors_SMD:R_0603_HandSoldering" V 2780 3600 50  0001 C CNN
-F 3 "~" H 2850 3600 50  0001 C CNN
+F 3 "https://akizukidenshi.com/catalog/g/gR-14122/" H 2850 3600 50  0001 C CNN
+F 4 "https://akizukidenshi.com/catalog/g/gR-14122/" H 2850 3600 50  0001 C CNN "Buy"
+F 5 "https://akizukidenshi.com/catalog/g/gR-14122/" H 2850 3600 50  0001 C CNN "Vendor"
 	1    2850 3600
 	0    1    1    0
@@
 F 1 "LED5" H 3143 3786 50  0000 C CNN
 F 2 "LEDs:LED_0603_HandSoldering" H 3150 3950 50  0001 C CNN
-F 3 "~" H 3150 3950 50  0001 C CNN
+F 3 "https://akizukidenshi.com/catalog/g/gI-11879/" H 3150 3950 50  0001 C CNN
+F 4 "https://akizukidenshi.com/catalog/g/gI-11879/" H 3150 3950 50  0001 C CNN "Buy"
+F 5 "https://akizukidenshi.com/catalog/g/gI-11879/" H 3150 3950 50  0001 C CNN "Vendor"
 	1    3150 3950
 	-1   0    0    1
@@
 F 1 "1k" V 2850 3950 50  0000 C CNN
 F 2 "Resistors_SMD:R_0603_HandSoldering" V 2780 3950 50  0001 C CNN
-F 3 "~" H 2850 3950 50  0001 C CNN
+F 3 "https://akizukidenshi.com/catalog/g/gR-14122/" H 2850 3950 50  0001 C CNN
+F 4 "https://akizukidenshi.com/catalog/g/gR-14122/" H 2850 3950 50  0001 C CNN "Buy"
+F 5 "https://akizukidenshi.com/catalog/g/gR-14122/" H 2850 3950 50  0001 C CNN "Vendor"
 	1    2850 3950
 	0    1    1    0
@@
 F 1 "SMT-0440" H 4920 2355 50  0000 L CNN
 F 2 "PUI_Audio:SMT-0440-S-R" H 4750 2250 50  0001 C CNN
-F 3 "~" H 4740 2400 50  0001 C CNN
+F 3 "https://www.digikey.jp/ja/products/detail/pui-audio-inc/SMT-0440-S-R/5113609" H 4740 2400 50  0001 C CNN
+F 4 "https://www.digikey.jp/ja/products/detail/pui-audio-inc/SMT-0440-S-R/5113609" H 4750 2450 50  0001 C CNN "Buy"
+F 5 "https://www.digikey.jp/ja/products/detail/pui-audio-inc/SMT-0440-S-R/5113609" H 4750 2450 50  0001 C CNN "Vendor"
 	1    4750 2450
 	1    0    0    -1
@@
 F 1 "IRFML8244" H 4641 3205 50  0000 L CNN
 F 2 "TO_SOT_Packages_SMD:SOT-23" H 4650 3350 50  0001 C CNN
-F 3 "~" H 4450 3250 50  0001 C CNN
+F 3 "https://akizukidenshi.com/catalog/g/gI-06051/" H 4450 3250 50  0001 C CNN
+F 4 "https://akizukidenshi.com/catalog/g/gI-06051/" H 4450 3250 50  0001 C CNN "Buy"
+F 5 "https://akizukidenshi.com/catalog/g/gI-06051/" H 4450 3250 50  0001 C CNN "Vendor"
 	1    4450 3250
 	1    0    0    -1
@@
 F 1 "1k" H 4620 2855 50  0000 L CNN
 F 2 "Resistors_SMD:R_0603_HandSoldering" V 4480 2900 50  0001 C CNN
-F 3 "~" H 4550 2900 50  0001 C CNN
+F 3 "https://akizukidenshi.com/catalog/g/gR-14122/" H 4550 2900 50  0001 C CNN
+F 4 "https://akizukidenshi.com/catalog/g/gR-14122/" H 4550 2900 50  0001 C CNN "Buy"
+F 5 "https://akizukidenshi.com/catalog/g/gR-14122/" H 4550 2900 50  0001 C CNN "Vendor"
 	1    4550 2900
 	1    0    0    -1
@@
 F 1 "1k" V 2850 4350 50  0000 C CNN
 F 2 "Resistors_SMD:R_0603_HandSoldering" V 2780 4350 50  0001 C CNN
-F 3 "~" H 2850 4350 50  0001 C CNN
+F 3 "https://akizukidenshi.com/catalog/g/gR-14122/" H 2850 4350 50  0001 C CNN
+F 4 "https://akizukidenshi.com/catalog/g/gR-14122/" H 2850 4350 50  0001 C CNN "Buy"
+F 5 "https://akizukidenshi.com/catalog/g/gR-14122/" H 2850 4350 50  0001 C CNN "Vendor"
 	1    2850 4350
 	0    1    1    0
@@
 F 1 "LED6" H 3143 4186 50  0000 C CNN
 F 2 "LEDs:LED_0603_HandSoldering" H 3150 4350 50  0001 C CNN
-F 3 "~" H 3150 4350 50  0001 C CNN
+F 3 "https://akizukidenshi.com/catalog/g/gI-11879/" H 3150 4350 50  0001 C CNN
+F 4 "https://akizukidenshi.com/catalog/g/gI-11879/" H 3150 4350 50  0001 C CNN "Buy"
+F 5 "https://akizukidenshi.com/catalog/g/gI-11879/" H 3150 4350 50  0001 C CNN "Vendor"
 	1    3150 4350
 	-1   0    0    1
@@
 F 1 "Button1" V 6795 3448 50  0000 L CNN
 F 2 "Buttons_Switches_SMD:SW_SPST_EVQP2" H 6750 3500 50  0001 C CNN
-F 3 "" H 6750 3500 50  0001 C CNN
+F 3 "https://akizukidenshi.com/catalog/g/gP-06185/" H 6750 3500 50  0001 C CNN
+F 4 "https://akizukidenshi.com/catalog/g/gP-06185/" H 6750 3300 50  0001 C CNN "Buy"
+F 5 "https://akizukidenshi.com/catalog/g/gP-06185/" H 6750 3300 50  0001 C CNN "Vendor"
 	1    6750 3300
 	0    1    1    0
@@
 F 1 "ButtonLED1" H 6343 3786 50  0000 C CNN
 F 2 "LEDs:LED_0603_HandSoldering" H 6350 3950 50  0001 C CNN
-F 3 "~" H 6350 3950 50  0001 C CNN
+F 3 "https://akizukidenshi.com/catalog/g/gI-11879/" H 6350 3950 50  0001 C CNN
+F 4 "https://akizukidenshi.com/catalog/g/gI-11879/" H 6350 3950 50  0001 C CNN "Buy"
+F 5 "https://akizukidenshi.com/catalog/g/gI-11879/" H 6350 3950 50  0001 C CNN "Vendor"
 	1    6350 3950
 	0    -1   -1   0
@@
 F 1 "1k" V 6350 3650 50  0000 C CNN
 F 2 "Resistors_SMD:R_0603_HandSoldering" V 6280 3650 50  0001 C CNN
-F 3 "~" H 6350 3650 50  0001 C CNN
+F 3 "https://akizukidenshi.com/catalog/g/gR-14122/" H 6350 3650 50  0001 C CNN
+F 4 "https://akizukidenshi.com/catalog/g/gR-14122/" H 6350 3650 50  0001 C CNN "Buy"
+F 5 "https://akizukidenshi.com/catalog/g/gR-14122/" H 6350 3650 50  0001 C CNN "Vendor"
 	1    6350 3650
 	-1   0    0    1
@@
 F 2 "Resistors_SMD:R_0603_HandSoldering" V 6680 3950 50  0001 C CNN
 F 3 "~" H 6750 3950 50  0001 C CNN
+F 4 "~" H 6750 3950 50  0001 C CNN "Buy"
+F 5 "~" H 6750 3950 50  0001 C CNN "Vendor"
 	1    6750 3950
 	-1   0    0    1
@@
 F 1 "Button2" V 7745 3448 50  0000 L CNN
 F 2 "Buttons_Switches_SMD:SW_SPST_EVQP2" H 7700 3500 50  0001 C CNN
-F 3 "" H 7700 3500 50  0001 C CNN
+F 3 "https://akizukidenshi.com/catalog/g/gP-06185/" H 7700 3500 50  0001 C CNN
+F 4 "https://akizukidenshi.com/catalog/g/gP-06185/" H 7700 3300 50  0001 C CNN "Buy"
+F 5 "https://akizukidenshi.com/catalog/g/gP-06185/" H 7700 3300 50  0001 C CNN "Vendor"
 	1    7700 3300
 	0    1    1    0
@@
 F 1 "ButtonLED2" H 7293 3786 50  0000 C CNN
 F 2 "LEDs:LED_0603_HandSoldering" H 7300 3950 50  0001 C CNN
-F 3 "~" H 7300 3950 50  0001 C CNN
+F 3 "https://akizukidenshi.com/catalog/g/gI-11879/" H 7300 3950 50  0001 C CNN
+F 4 "https://akizukidenshi.com/catalog/g/gI-11879/" H 7300 3950 50  0001 C CNN "Buy"
+F 5 "https://akizukidenshi.com/catalog/g/gI-11879/" H 7300 3950 50  0001 C CNN "Vendor"
 	1    7300 3950
 	0    -1   -1   0
@@
 F 1 "1k" V 7300 3650 50  0000 C CNN
 F 2 "Resistors_SMD:R_0603_HandSoldering" V 7230 3650 50  0001 C CNN
-F 3 "~" H 7300 3650 50  0001 C CNN
+F 3 "https://akizukidenshi.com/catalog/g/gR-14122/" H 7300 3650 50  0001 C CNN
+F 4 "https://akizukidenshi.com/catalog/g/gR-14122/" H 7300 3650 50  0001 C CNN "Buy"
+F 5 "https://akizukidenshi.com/catalog/g/gR-14122/" H 7300 3650 50  0001 C CNN "Vendor"
 	1    7300 3650
 	-1   0    0    1
@@
 F 2 "Resistors_SMD:R_0603_HandSoldering" V 7630 3950 50  0001 C CNN
 F 3 "~" H 7700 3950 50  0001 C CNN
+F 4 "~" H 7700 3950 50  0001 C CNN "Buy"
+F 5 "~" H 7700 3950 50  0001 C CNN "Vendor"
 	1    7700 3950
 	-1   0    0    1
