File: pcb/MicroController.sch (KiCad schematic (older format))
At the start: 2 parts, among them J8 CN2_Right, J9 CN1_Left

Commit message: Make netlist
Parts:
- J8, J9: footprint (none) -> Pin_Headers:Pin_Header_Straight_2x13_Pitch2.54mm
Connections:
- net Button1: now reaches J9.15 (Pin_15)
- net Button2: now reaches J9.16 (Pin_16)
- no-connect marks 17 -> 15
Changed lines of the file:
@@
 F 0 "J9" H 4500 2817 50  0000 C CNN
 F 1 "CN1_Left" H 4500 2726 50  0000 C CNN
-F 2 "" H 4450 2000 50  0001 C CNN
+F 2 "Pin_Headers:Pin_Header_Straight_2x13_Pitch2.54mm" H 4450 2000 50  0001 C CNN
 F 3 "~" H 4450 2000 50  0001 C CNN
 	1    4450 2000
@@
 F 0 "J8" H 1750 2767 50  0000 C CNN
 F 1 "CN2_Right" H 1750 2676 50  0000 C CNN
-F 2 "" H 1700 1950 50  0001 C CNN
+F 2 "Pin_Headers:Pin_Header_Straight_2x13_Pitch2.54mm" H 1700 1950 50  0001 C CNN
 F 3 "~" H 1700 1950 50  0001 C CNN
 	1    1700 1950
@@
 TIM2 EncoderL\nTIM4 Motor\nTIM8 EncoderR\nTIM9(TIM5) IR\nTIM12 BUZZER
 NoConn ~ 4750 1900
-NoConn ~ 4750 2100
-NoConn ~ 4250 2100
 NoConn ~ 4250 1900
+Text HLabel 4250 2100 0    50   Input ~ 0
+Button1
+Text HLabel 4750 2100 2    50   Input ~ 0
+Button2
 $EndSCHEMATC

Commit message: Update schematic
Parts:
- removed J8: CN2_Right, Pin_Headers:Pin_Header_Straight_2x13_Pitch2.54mm, symbol Connector_Generic:Conn_02x13_Odd_Even
- removed J9: CN1_Left, Pin_Headers:Pin_Header_Straight_2x13_Pitch2.54mm, symbol Connector_Generic:Conn_02x13_Odd_Even
- added J7: STM32F405Board, Zero_Module:STM32F405Board, symbol Connector_Generic:Conn_02x26_Odd_Even
Connections:
- net +3V3: now also J7.2 (Pin_2), J7.28 (Pin_28)
- net BAT_REF: now also J7.7 (Pin_7)
- net Button1: now also J7.15 (Pin_15)
- net Button2: now also J7.16 (Pin_16)
- net Buzzer: now also J7.52 (Pin_52)
- net GND: now also J7.1 (Pin_1), J7.27 (Pin_27)
- net IMU_CLK: now also J7.34 (Pin_34)
- net IMU_CS: now also J7.33 (Pin_33)
- net IMU_MISO: now also J7.35 (Pin_35)
- net IMU_MOSI: now also J7.36 (Pin_36)
- net IR_Sensor_IN1: now also J7.3 (Pin_3)
- net IR_Sensor_IN2: now also J7.4 (Pin_4)
- net IR_Sensor_IN3: now also J7.5 (Pin_5)
- net IR_Sensor_IN4: now also J7.6 (Pin_6)
- net IR_Sensor_OUT1: now also J7.31 (Pin_31)
- net IR_Sensor_OUT2: now also J7.32 (Pin_32)
- net LED1: now also J7.17 (Pin_17)
- net LED2: now also J7.18 (Pin_18)
- net LED3: now also J7.19 (Pin_19)
- net LED4: now also J7.20 (Pin_20)
- net LED5: now also J7.21 (Pin_21)
- net LED6: now also J7.22 (Pin_22)
- net Left_EncoderA: now also J7.29 (Pin_29)
- net Left_EncoderB: now also J7.30 (Pin_30)
- net Left_Motor_OUT1: now also J7.45 (Pin_45)
- net Left_Motor_OUT2: now also J7.46 (Pin_46)
- net NRST: now also J7.26 (Pin_26)
- net Right_EncoderA: now also J7.9 (Pin_9)
- net Right_EncoderB: now also J7.10 (Pin_10)
- net Right_Motor_OUT1: now also J7.23 (Pin_23)
- net Right_Motor_OUT2: now also J7.24 (Pin_24)
- net SWCLK: now also J7.43 (Pin_43)
- net SWDIO: now also J7.42 (Pin_42)
- net UART_RX: now also J7.14 (Pin_14)
- net UART_TX: now also J7.13 (Pin_13)
Other:
- note added: "CN1(Left)\n--------------------------------------------\nCN2(Right)"
Changed lines of the file:
@@
 Comment4 ""
 $EndDescr
-$Comp
-L Connector_Generic:Conn_02x13_Odd_Even J9
-U 1 1 61651D0A
-P 4450 2000
-F 0 "J9" H 4500 2817 50  0000 C CNN
-F 1 "CN1_Left" H 4500 2726 50  0000 C CNN
-F 2 "Pin_Headers:Pin_Header_Straight_2x13_Pitch2.54mm" H 4450 2000 50  0001 C CNN
-F 3 "~" H 4450 2000 50  0001 C CNN
-	1    4450 2000
-	1    0    0    -1
-$EndComp
-$Comp
-L Connector_Generic:Conn_02x13_Odd_Even J8
-U 1 1 61652D70
-P 1700 1950
-F 0 "J8" H 1750 2767 50  0000 C CNN
-F 1 "CN2_Right" H 1750 2676 50  0000 C CNN
-F 2 "Pin_Headers:Pin_Header_Straight_2x13_Pitch2.54mm" H 1700 1950 50  0001 C CNN
-F 3 "~" H 1700 1950 50  0001 C CNN
-	1    1700 1950
-	1    0    0    -1
-$EndComp
 Text Notes 3300 2600 0    63   ~ 0
 GND\nPC0\nPC2\nPC4\nPC6\nPC8\nPC10\nPC12\nPB0\nPB2\nPB4\nPB6\nVBAT
 Text Notes 5500 2650 0    63   ~ 0
 VDD\nPC1\nPC3\nPC5\nPC7\nPC9\nPC11\nPC13\nPB1\nPB3\nPB5\nPB7\nRESET
-Text Notes 2700 2600 0    63   ~ 0
-VDD\nPA1\nPA3\nPA5\nPA7\nPA9\nPA11\nPA13\nPA15\nPB9\nPB11\nPB13\nPB15
-Text Notes 550  2600 0    63   ~ 0
-GND\nPA0\nPA2\nPA4\nPA6\nPA8\nPA10\nPA12\nPA14\nPB8\nPB10\nPB12\nPB14
-$Comp
-L power:GND #PWR044
-U 1 1 616799E3
-P 1500 1350
-F 0 "#PWR044" H 1500 1100 50  0001 C CNN
-F 1 "GND" V 1505 1222 50  0000 R CNN
-F 2 "" H 1500 1350 50  0001 C CNN
-F 3 "" H 1500 1350 50  0001 C CNN
-	1    1500 1350
-	0    1    1    0
-$EndComp
 $Comp
 L power:GND #PWR046
@@
 F 3 "" H 4250 1400 50  0001 C CNN
 	1    4250 1400
-	0    1    1    0
-$EndComp
-$Comp
-L power:+3.3V #PWR045
-U 1 1 6167CB5D
-P 2000 1350
-F 0 "#PWR045" H 2000 1200 50  0001 C CNN
-F 1 "+3.3V" V 2015 1478 50  0000 L CNN
-F 2 "" H 2000 1350 50  0001 C CNN
-F 3 "" H 2000 1350 50  0001 C CNN
-	1    2000 1350
 	0    1    1    0
 $EndComp
@@
 Text HLabel 4750 2400 2    50   Output ~ 0
 LED6
-Text HLabel 1500 1650 0    50   Output ~ 0
-IMU_CS
-Text HLabel 1500 1750 0    50   Input ~ 0
-IMU_MISO
-Text HLabel 2000 1750 2    50   Output ~ 0
-IMU_MOSI
-Text HLabel 2000 1650 2    50   Output ~ 0
-IMU_CLK
 Text HLabel 4250 2000 0    50   Output ~ 0
 UART_TX
 Text HLabel 4750 2000 2    50   Input ~ 0
 UART_RX
-Text HLabel 2000 2050 2    50   BiDi ~ 0
-SWDIO
-Text HLabel 1500 2150 0    50   Input ~ 0
-SWCLK
 Text HLabel 4750 2600 2    50   Input ~ 0
 NRST
@@
 Text HLabel 4750 1800 2    50   Input ~ 0
 Right_EncoderB
-Text HLabel 1500 1450 0    50   Input ~ 0
-Left_EncoderA
-Text HLabel 2000 1450 2    50   Input ~ 0
-Left_EncoderB
-NoConn ~ 1500 2350
 NoConn ~ 4250 2600
-NoConn ~ 2000 2350
-NoConn ~ 1500 1850
-NoConn ~ 1500 1950
-NoConn ~ 1500 2050
-NoConn ~ 2000 1850
-NoConn ~ 2000 1950
-NoConn ~ 2000 2150
 Text HLabel 4250 2500 0    50   Input ~ 0
 Right_Motor_OUT1
 Text HLabel 4750 2500 2    50   Input ~ 0
 Right_Motor_OUT2
-Text HLabel 1500 2250 0    50   Input ~ 0
-Left_Motor_OUT1
-Text HLabel 2000 2250 2    50   Input ~ 0
-Left_Motor_OUT2
 NoConn ~ 4750 1700
-Text HLabel 2000 2550 2    50   Output ~ 0
-Buzzer
-NoConn ~ 2000 2450
-NoConn ~ 1500 2450
-NoConn ~ 1500 2550
-Text HLabel 1500 1550 0    50   Output ~ 0
-IR_Sensor_OUT1
-Text HLabel 2000 1550 2    50   Output ~ 0
-IR_Sensor_OUT2
-Text Notes 1500 3700 0    100  ~ 20
-TIM2 EncoderL\nTIM4 Motor\nTIM8 EncoderR\nTIM9(TIM5) IR\nTIM12 BUZZER
 NoConn ~ 4750 1900
 NoConn ~ 4250 1900
@@
 Text HLabel 4750 2100 2    50   Input ~ 0
 Button2
+Text Notes 1500 4500 0    100  ~ 20
+TIM2 EncoderL\nTIM4 Motor\nTIM8 EncoderR\nTIM9(TIM5) IR\nTIM12 BUZZER
+Text Notes 3300 3950 0    63   ~ 0
+GND\nPA0\nPA2\nPA4\nPA6\nPA8\nPA10\nPA12\nPA14\nPB8\nPB10\nPB12\nPB14
+$Comp
+L power:GND #PWR044
+U 1 1 616799E3
+P 4250 2700
+F 0 "#PWR044" H 4250 2450 50  0001 C CNN
+F 1 "GND" V 4255 2572 50  0000 R CNN
+F 2 "" H 4250 2700 50  0001 C CNN
+F 3 "" H 4250 2700 50  0001 C CNN
+	1    4250 2700
+	0    1    1    0
+$EndComp
+$Comp
+L power:+3.3V #PWR045
+U 1 1 6167CB5D
+P 4750 2700
+F 0 "#PWR045" H 4750 2550 50  0001 C CNN
+F 1 "+3.3V" V 4765 2828 50  0000 L CNN
+F 2 "" H 4750 2700 50  0001 C CNN
+F 3 "" H 4750 2700 50  0001 C CNN
+	1    4750 2700
+	0    1    1    0
+$EndComp
+Text HLabel 4250 3000 0    50   Output ~ 0
+IMU_CS
+Text HLabel 4250 3100 0    50   Input ~ 0
+IMU_MISO
+Text HLabel 4750 3100 2    50   Output ~ 0
+IMU_MOSI
+Text HLabel 4750 3000 2    50   Output ~ 0
+IMU_CLK
+Text HLabel 4750 3400 2    50   BiDi ~ 0
+SWDIO
+Text HLabel 4250 3500 0    50   Input ~ 0
+SWCLK
+Text HLabel 4250 2800 0    50   Input ~ 0
+Left_EncoderA
+Text HLabel 4750 2800 2    50   Input ~ 0
+Left_EncoderB
+NoConn ~ 4250 3700
+NoConn ~ 4750 3700
+NoConn ~ 4250 3200
+NoConn ~ 4250 3300
+NoConn ~ 4250 3400
+NoConn ~ 4750 3200
+NoConn ~ 4750 3300
+NoConn ~ 4750 3500
+Text HLabel 4250 3600 0    50   Input ~ 0
+Left_Motor_OUT1
+Text HLabel 4750 3600 2    50   Input ~ 0
+Left_Motor_OUT2
+Text HLabel 4750 3900 2    50   Output ~ 0
+Buzzer
+NoConn ~ 4750 3800
+NoConn ~ 4250 3800
+NoConn ~ 4250 3900
+Text HLabel 4250 2900 0    50   Output ~ 0
+IR_Sensor_OUT1
+Text HLabel 4750 2900 2    50   Output ~ 0
+IR_Sensor_OUT2
+Text Notes 5500 3950 0    63   ~ 0
+VDD\nPA1\nPA3\nPA5\nPA7\nPA9\nPA11\nPA13\nPA15\nPB9\nPB11\nPB13\nPB15
+$Comp
+L Connector_Generic:Conn_02x26_Odd_Even J7
+U 1 1 616EAB41
+P 4450 2600
+F 0 "J7" H 4500 4017 50  0000 C CNN
+F 1 "STM32F405Board" H 4500 3926 50  0000 C CNN
+F 2 "Zero_Module:STM32F405Board" H 4450 2600 50  0001 C CNN
+F 3 "~" H 4450 2600 50  0001 C CNN
+	1    4450 2600
+	1    0    0    -1
+$EndComp
+Text Notes 2150 2700 0    39   ~ 0
+CN1(Left)\n--------------------------------------------\nCN2(Right)
 $EndSCHEMATC

Commit message: Update pcb
Connections:
- net +3V3: now also J7.25 (Pin_25)
- no-connect marks 15 -> 14
Changed lines of the file:
@@
 Text HLabel 4750 2200 2    50   Output ~ 0
 LED2
-Text HLabel 4750 2300 2    50   Output ~ 0
-LED4
 Text HLabel 4250 2300 0    50   Output ~ 0
 LED3
-Text HLabel 4250 2400 0    50   Output ~ 0
-LED5
-Text HLabel 4750 2400 2    50   Output ~ 0
-LED6
 Text HLabel 4250 2000 0    50   Output ~ 0
 UART_TX
@@
 Text HLabel 4750 1800 2    50   Input ~ 0
 Right_EncoderB
-NoConn ~ 4250 2600
 Text HLabel 4250 2500 0    50   Input ~ 0
 Right_Motor_OUT1
@@
 Text HLabel 4750 3100 2    50   Output ~ 0
 IMU_MOSI
-Text HLabel 4750 3000 2    50   Output ~ 0
-IMU_CLK
 Text HLabel 4750 3400 2    50   BiDi ~ 0
 SWDIO
 Text HLabel 4250 3500 0    50   Input ~ 0
 SWCLK
-Text HLabel 4250 2800 0    50   Input ~ 0
-Left_EncoderA
 Text HLabel 4750 2800 2    50   Input ~ 0
 Left_EncoderB
@@
 Text HLabel 4750 3900 2    50   Output ~ 0
 Buzzer
-NoConn ~ 4750 3800
-NoConn ~ 4250 3800
 NoConn ~ 4250 3900
 Text HLabel 4250 2900 0    50   Output ~ 0
@@
 	1    0    0    -1
 $EndComp
-Text Notes 2150 2700 0    39   ~ 0
+$Comp
+L power:+3.3V #PWR054
+U 1 1 617FE91D
+P 4250 2600
+F 0 "#PWR054" H 4250 2450 50  0001 C CNN
+F 1 "+3.3V" V 4265 2728 50  0000 L CNN
+F 2 "" H 4250 2600 50  0001 C CNN
+F 3 "" H 4250 2600 50  0001 C CNN
+	1    4250 2600
+	0    -1   -1   0
+$EndComp
+NoConn ~ 4750 3800
+NoConn ~ 4250 3800
+Text HLabel 4250 2400 0    50   Output ~ 0
+LED5
+Text HLabel 4750 2400 2    50   Output ~ 0
+LED6
+Text HLabel 4750 2300 2    50   Output ~ 0
+LED4
+Text HLabel 4750 3000 2    50   Output ~ 0
+IMU_CLK
+Text HLabel 4250 2800 0    50   Input ~ 0
+Left_EncoderA
+Text Notes 2050 2700 0    39   ~ 0
 CN1(Left)\n--------------------------------------------\nCN2(Right)
 $EndSCHEMATC

Commit message: Write about where to buy the parts
Parts:
- J7: Buy (none) -> https://strawberry-linux.com/catalog/items?code=32405; Vendor (none) -> https://strawberry-linux.com/catalog/items?code=32405
Changed lines of the file:
@@
 F 1 "STM32F405Board" H 4500 3926 50  0000 C CNN
 F 2 "Zero_Module:STM32F405Board" H 4450 2600 50  0001 C CNN
-F 3 "~" H 4450 2600 50  0001 C CNN
+F 3 "https://strawberry-linux.com/catalog/items?code=32405" H 4450 2600 50  0001 C CNN
+F 4 "https://strawberry-linux.com/catalog/items?code=32405" H 4450 2600 50  0001 C CNN "Buy"
+F 5 "https://strawberry-linux.com/catalog/items?code=32405" H 4450 2600 50  0001 C CNN "Vendor"
 	1    4450 2600
 	1    0    0    -1
