File: pcb/Motor.sch (KiCad schematic (older format))
At the start: 5 parts

Commit message: Finish the schematic
Parts:
- gave numbers to parts that had none: 5
Connections:
- net Left_Encoder_A renamed Left_EncoderA
- net Left_Encoder_B renamed Left_EncoderB
- net Left_Motor_OUT_A renamed Left_Motor_OUT1
- net Left_Motor_OUT_B renamed Left_Motor_OUT2
- net Right_Encoder_A renamed Right_EncoderA
- net Right_Encoder_B renamed Right_EncoderB
- net Right_Motor_OUT_A renamed Right_Motor_OUT1
- net Right_Motor_OUT_B renamed Right_Motor_OUT2
Changed lines of the file:
@@
 $Descr A4 11693 8268
 encoding utf-8
-Sheet 4 5
+Sheet 3 8
 Title ""
 Date ""
@@
 $EndDescr
 $Comp
-L REF1933:DRV8835 U?
+L REF1933:DRV8835 U7
 U 1 1 61358D09
 P 2450 4000
-F 0 "U?" H 2200 4450 60  0000 C CNN
+F 0 "U7" H 2200 4450 60  0000 C CNN
 F 1 "DRV8835" H 2150 4350 60  0000 C CNN
 F 2 "" H 1400 4200 60  0000 C CNN
@@
 $EndComp
 $Comp
-L Connector:Conn_01x06_Female J?
+L Connector:Conn_01x06_Female J4
 U 1 1 61359DC6
 P 4950 4350
-F 0 "J?" H 4978 4326 50  0000 L CNN
+F 0 "J4" H 4978 4326 50  0000 L CNN
 F 1 "Left_Motor" H 4978 4235 50  0000 L CNN
 F 2 "" H 4950 4350 50  0001 C CNN
@@
 $EndComp
 $Comp
-L Connector:Conn_01x06_Female J?
+L Connector:Conn_01x06_Female J5
 U 1 1 6135AD13
 P 4950 5150
-F 0 "J?" H 4978 5126 50  0000 L CNN
+F 0 "J5" H 4978 5126 50  0000 L CNN
 F 1 "Right_Motor" H 4978 5035 50  0000 L CNN
 F 2 "" H 4950 5150 50  0001 C CNN
@@
 $EndComp
 $Comp
-L power:+3.3V #PWR?
+L power:+3.3V #PWR0104
 U 1 1 6135BC63
 P 2400 3400
-F 0 "#PWR?" H 2400 3250 50  0001 C CNN
+F 0 "#PWR0104" H 2400 3250 50  0001 C CNN
 F 1 "+3.3V" H 2250 3400 50  0000 C CNN
 F 2 "" H 2400 3400 50  0001 C CNN
@@
 $EndComp
 $Comp
-L power:+BATT #PWR?
+L power:+BATT #PWR0105
 U 1 1 6135D44B
 P 2500 3250
-F 0 "#PWR?" H 2500 3100 50  0001 C CNN
+F 0 "#PWR0105" H 2500 3100 50  0001 C CNN
 F 1 "+BATT" H 2650 3250 50  0000 C CNN
 F 2 "" H 2500 3250 50  0001 C CNN
@@
 $EndComp
 $Comp
-L power:GND #PWR?
+L power:GND #PWR0106
 U 1 1 6135DF52
 P 4750 4650
-F 0 "#PWR?" H 4750 4400 50  0001 C CNN
+F 0 "#PWR0106" H 4750 4400 50  0001 C CNN
 F 1 "GND" V 4755 4522 50  0000 R CNN
 F 2 "" H 4750 4650 50  0001 C CNN
@@
 $EndComp
 $Comp
-L power:GND #PWR?
+L power:GND #PWR0107
 U 1 1 6135E108
 P 4750 5450
-F 0 "#PWR?" H 4750 5200 50  0001 C CNN
+F 0 "#PWR0107" H 4750 5200 50  0001 C CNN
 F 1 "GND" V 4755 5322 50  0000 R CNN
 F 2 "" H 4750 5450 50  0001 C CNN
@@
 $EndComp
 $Comp
-L power:+3.3V #PWR?
+L power:+3.3V #PWR0108
 U 1 1 6135E5C7
 P 4750 5150
-F 0 "#PWR?" H 4750 5000 50  0001 C CNN
+F 0 "#PWR0108" H 4750 5000 50  0001 C CNN
 F 1 "+3.3V" V 4750 5400 50  0000 C CNN
 F 2 "" H 4750 5150 50  0001 C CNN
@@
 $EndComp
 $Comp
-L power:+3.3V #PWR?
+L power:+3.3V #PWR0109
 U 1 1 6135F604
 P 4750 4350
-F 0 "#PWR?" H 4750 4200 50  0001 C CNN
+F 0 "#PWR0109" H 4750 4200 50  0001 C CNN
 F 1 "+3.3V" V 4750 4600 50  0000 C CNN
 F 2 "" H 4750 4350 50  0001 C CNN
@@
 	0    -1   -1   0
 $EndComp
-Text HLabel 4750 4450 0    50   Output ~ 0
-Left_Encoder_A
 Text HLabel 4750 4550 0    50   Output ~ 0
-Left_Encoder_B
+Left_EncoderB
 Text HLabel 4750 5250 0    50   Output ~ 0
-Right_Encoder_A
-Text HLabel 4750 5350 0    50   Output ~ 0
-Right_Encoder_B
-$Comp
-L power:GND #PWR?
+Right_EncoderA
+$Comp
+L power:GND #PWR0110
 U 1 1 61367EC5
 P 2400 4450
-F 0 "#PWR?" H 2400 4200 50  0001 C CNN
+F 0 "#PWR0110" H 2400 4200 50  0001 C CNN
 F 1 "GND" H 2405 4277 50  0000 C CNN
 F 2 "" H 2400 4450 50  0001 C CNN
@@
 	2000 4450 2400 4450
 $Comp
-L Device:C C?
+L Device:C C13
 U 1 1 61368A7C
 P 1100 4300
-F 0 "C?" H 1150 4400 50  0000 L CNN
+F 0 "C13" H 1150 4400 50  0000 L CNN
 F 1 "22u" H 1150 4200 50  0000 L CNN
 F 2 "" H 1138 4150 50  0001 C CNN
@@
 $EndComp
 $Comp
-L Device:C C?
+L Device:C C12
 U 1 1 61369106
 P 800 4300
-F 0 "C?" H 850 4400 50  0000 L CNN
+F 0 "C12" H 850 4400 50  0000 L CNN
 F 1 "0.1u" H 850 4200 50  0000 L CNN
 F 2 "" H 838 4150 50  0001 C CNN
@@
 	2400 3400 2400 3650
 Text HLabel 2000 3800 0    50   Input ~ 0
-Left_Motor_OUT_A
+Left_Motor_OUT1
 Text HLabel 2000 3900 0    50   Input ~ 0
-Left_Motor_OUT_B
+Left_Motor_OUT2
 Text HLabel 2000 4050 0    50   Input ~ 0
-Right_Motor_OUT_A
+Right_Motor_OUT1
 Text HLabel 2000 4150 0    50   Input ~ 0
-Right_Motor_OUT_B
-$Comp
-L power:GND #PWR?
+Right_Motor_OUT2
+$Comp
+L power:GND #PWR0111
 U 1 1 613823C3
 P 800 4450
-F 0 "#PWR?" H 800 4200 50  0001 C CNN
+F 0 "#PWR0111" H 800 4200 50  0001 C CNN
 F 1 "GND" H 805 4277 50  0000 C CNN
 F 2 "" H 800 4450 50  0001 C CNN
@@
 	800  4150 1100 4150
 $Comp
-L power:+BATT #PWR?
+L power:+BATT #PWR0112
 U 1 1 61383160
 P 800 4150
-F 0 "#PWR?" H 800 4000 50  0001 C CNN
+F 0 "#PWR0112" H 800 4000 50  0001 C CNN
 F 1 "+BATT" H 815 4323 50  0000 C CNN
 F 2 "" H 800 4150 50  0001 C CNN
@@
 Wire Wire Line
 	4000 4200 2900 4200
+Text HLabel 4750 4450 0    50   Output ~ 0
+Left_EncoderA
+Text HLabel 4750 5350 0    50   Output ~ 0
+Right_EncoderB
 $EndSCHEMATC

Commit message: Make netlist
Parts:
- removed U7: DRV8835, symbol REF1933:DRV8835
- added J12: DRV8835_Left, Pin_Headers:Pin_Header_Straight_1x06_Pitch2.54mm, symbol Connector:Conn_01x06_Male
- added J13: DRV8835_Right, Pin_Headers:Pin_Header_Straight_1x06_Pitch2.54mm, symbol Connector:Conn_01x06_Male
- C12, C13: footprint (none) -> Capacitors_SMD:C_0603_HandSoldering
- J4, J5: footprint (none) -> Connector_JST:JST_XH_B6B-XH-AM_1x06_P2.50mm_Vertical
Connections:
- net +3V3: now also J13.1 (Pin_1)
- net +BATT: now also J12.1 (Pin_1)
- net GND: now also J12.6 (Pin_6), J13.2 (Pin_2)
- net Left_Motor_OUT1: now also J13.3 (Pin_3)
- net Left_Motor_OUT2: now also J13.4 (Pin_4)
- net Right_Motor_OUT1: now also J13.5 (Pin_5)
- net Right_Motor_OUT2: now also J13.6 (Pin_6)
- net at J4.1 (Pin_1): now also J12.3 (Pin_3)
- net at J4.2 (Pin_2): now also J12.2 (Pin_2)
- net at J5.1 (Pin_1): now also J12.5 (Pin_5)
- net at J5.2 (Pin_2): now also J12.4 (Pin_4)
Other:
- moved on the sheet: J4, J5
Changed lines of the file:
@@
 $EndDescr
-$Comp
-L REF1933:DRV8835 U7
-U 1 1 61358D09
-P 2450 4000
-F 0 "U7" H 2200 4450 60  0000 C CNN
-F 1 "DRV8835" H 2150 4350 60  0000 C CNN
-F 2 "" H 1400 4200 60  0000 C CNN
-F 3 "" H 1400 4200 60  0000 C CNN
-	1    2450 4000
-	1    0    0    -1
-$EndComp
-$Comp
-L Connector:Conn_01x06_Female J4
-U 1 1 61359DC6
-P 4950 4350
-F 0 "J4" H 4978 4326 50  0000 L CNN
-F 1 "Left_Motor" H 4978 4235 50  0000 L CNN
-F 2 "" H 4950 4350 50  0001 C CNN
-F 3 "~" H 4950 4350 50  0001 C CNN
-	1    4950 4350
-	1    0    0    -1
-$EndComp
-$Comp
-L Connector:Conn_01x06_Female J5
-U 1 1 6135AD13
-P 4950 5150
-F 0 "J5" H 4978 5126 50  0000 L CNN
-F 1 "Right_Motor" H 4978 5035 50  0000 L CNN
-F 2 "" H 4950 5150 50  0001 C CNN
-F 3 "~" H 4950 5150 50  0001 C CNN
-	1    4950 5150
-	1    0    0    -1
-$EndComp
 $Comp
 L power:+3.3V #PWR0104
 U 1 1 6135BC63
-P 2400 3400
-F 0 "#PWR0104" H 2400 3250 50  0001 C CNN
-F 1 "+3.3V" H 2250 3400 50  0000 C CNN
-F 2 "" H 2400 3400 50  0001 C CNN
-F 3 "" H 2400 3400 50  0001 C CNN
-	1    2400 3400
-	1    0    0    -1
+P 3650 1700
+F 0 "#PWR0104" H 3650 1550 50  0001 C CNN
+F 1 "+3.3V" V 3550 1700 50  0000 C CNN
+F 2 "" H 3650 1700 50  0001 C CNN
+F 3 "" H 3650 1700 50  0001 C CNN
+	1    3650 1700
+	0    1    1    0
 $EndComp
 $Comp
 L power:+BATT #PWR0105
 U 1 1 6135D44B
-P 2500 3250
-F 0 "#PWR0105" H 2500 3100 50  0001 C CNN
-F 1 "+BATT" H 2650 3250 50  0000 C CNN
-F 2 "" H 2500 3250 50  0001 C CNN
-F 3 "" H 2500 3250 50  0001 C CNN
-	1    2500 3250
-	1    0    0    -1
+P 2200 1700
+F 0 "#PWR0105" H 2200 1550 50  0001 C CNN
+F 1 "+BATT" V 2300 1700 50  0000 C CNN
+F 2 "" H 2200 1700 50  0001 C CNN
+F 3 "" H 2200 1700 50  0001 C CNN
+	1    2200 1700
+	0    -1   -1   0
 $EndComp
 $Comp
 L power:GND #PWR0106
 U 1 1 6135DF52
-P 4750 4650
-F 0 "#PWR0106" H 4750 4400 50  0001 C CNN
-F 1 "GND" V 4755 4522 50  0000 R CNN
-F 2 "" H 4750 4650 50  0001 C CNN
-F 3 "" H 4750 4650 50  0001 C CNN
-	1    4750 4650
-	0    1    1    0
+P 1250 2150
+F 0 "#PWR0106" H 1250 1900 50  0001 C CNN
+F 1 "GND" V 1255 2022 50  0000 R CNN
+F 2 "" H 1250 2150 50  0001 C CNN
+F 3 "" H 1250 2150 50  0001 C CNN
+	1    1250 2150
+	0    -1   -1   0
 $EndComp
 $Comp
 L power:GND #PWR0107
 U 1 1 6135E108
-P 4750 5450
-F 0 "#PWR0107" H 4750 5200 50  0001 C CNN
-F 1 "GND" V 4755 5322 50  0000 R CNN
-F 2 "" H 4750 5450 50  0001 C CNN
-F 3 "" H 4750 5450 50  0001 C CNN
-	1    4750 5450
-	0    1    1    0
+P 1250 1400
+F 0 "#PWR0107" H 1250 1150 50  0001 C CNN
+F 1 "GND" V 1255 1272 50  0000 R CNN
+F 2 "" H 1250 1400 50  0001 C CNN
+F 3 "" H 1250 1400 50  0001 C CNN
+	1    1250 1400
+	0    -1   -1   0
 $EndComp
 $Comp
 L power:+3.3V #PWR0108
 U 1 1 6135E5C7
-P 4750 5150
-F 0 "#PWR0108" H 4750 5000 50  0001 C CNN
-F 1 "+3.3V" V 4750 5400 50  0000 C CNN
-F 2 "" H 4750 5150 50  0001 C CNN
-F 3 "" H 4750 5150 50  0001 C CNN
-	1    4750 5150
-	0    -1   -1   0
+P 1250 1700
+F 0 "#PWR0108" H 1250 1550 50  0001 C CNN
+F 1 "+3.3V" V 1250 1950 50  0000 C CNN
+F 2 "" H 1250 1700 50  0001 C CNN
+F 3 "" H 1250 1700 50  0001 C CNN
+	1    1250 1700
+	0    1    1    0
 $EndComp
 $Comp
 L power:+3.3V #PWR0109
 U 1 1 6135F604
-P 4750 4350
-F 0 "#PWR0109" H 4750 4200 50  0001 C CNN
-F 1 "+3.3V" V 4750 4600 50  0000 C CNN
-F 2 "" H 4750 4350 50  0001 C CNN
-F 3 "" H 4750 4350 50  0001 C CNN
-	1    4750 4350
-	0    -1   -1   0
-$EndComp
-Text HLabel 4750 4550 0    50   Output ~ 0
+P 1250 2450
+F 0 "#PWR0109" H 1250 2300 50  0001 C CNN
+F 1 "+3.3V" V 1250 2700 50  0000 C CNN
+F 2 "" H 1250 2450 50  0001 C CNN
+F 3 "" H 1250 2450 50  0001 C CNN
+	1    1250 2450
+	0    1    1    0
+$EndComp
+Text HLabel 1250 1500 2    50   Output ~ 0
 Left_EncoderB
-Text HLabel 4750 5250 0    50   Output ~ 0
+Text HLabel 1250 2350 2    50   Output ~ 0
 Right_EncoderA
-$Comp
-L power:GND #PWR0110
-U 1 1 61367EC5
-P 2400 4450
-F 0 "#PWR0110" H 2400 4200 50  0001 C CNN
-F 1 "GND" H 2405 4277 50  0000 C CNN
-F 2 "" H 2400 4450 50  0001 C CNN
-F 3 "" H 2400 4450 50  0001 C CNN
-	1    2400 4450
-	1    0    0    -1
-$EndComp
-Wire Wire Line
-	2400 4450 2500 4450
-Connection ~ 2400 4450
-Wire Wire Line
-	2000 4300 2000 4450
-Wire Wire Line
-	2000 4450 2400 4450
 $Comp
 L Device:C C13
@@
 F 0 "C13" H 1150 4400 50  0000 L CNN
 F 1 "22u" H 1150 4200 50  0000 L CNN
-F 2 "" H 1138 4150 50  0001 C CNN
+F 2 "Capacitors_SMD:C_0603_HandSoldering" H 1138 4150 50  0001 C CNN
 F 3 "~" H 1100 4300 50  0001 C CNN
 	1    1100 4300
@@
 F 0 "C12" H 850 4400 50  0000 L CNN
 F 1 "0.1u" H 850 4200 50  0000 L CNN
-F 2 "" H 838 4150 50  0001 C CNN
+F 2 "Capacitors_SMD:C_0603_HandSoldering" H 838 4150 50  0001 C CNN
 F 3 "~" H 800 4300 50  0001 C CNN
 	1    800  4300
 	1    0    0    -1
 $EndComp
-Wire Wire Line
-	2500 3250 2500 3650
-Wire Wire Line
-	2400 3400 2400 3650
-Text HLabel 2000 3800 0    50   Input ~ 0
+Text HLabel 3350 1900 2    50   Input ~ 0
 Left_Motor_OUT1
-Text HLabel 2000 3900 0    50   Input ~ 0
+Text HLabel 3350 2000 2    50   Input ~ 0
 Left_Motor_OUT2
-Text HLabel 2000 4050 0    50   Input ~ 0
+Text HLabel 3350 2100 2    50   Input ~ 0
 Right_Motor_OUT1
-Text HLabel 2000 4150 0    50   Input ~ 0
+Text HLabel 3350 2200 2    50   Input ~ 0
 Right_Motor_OUT2
 $Comp
@@
 $EndComp
 Connection ~ 800  4150
-Wire Wire Line
-	2900 3850 4750 3850
-Wire Wire Line
-	4750 3850 4750 4150
-Wire Wire Line
-	2900 3950 4600 3950
-Wire Wire Line
-	4600 3950 4600 4250
-Wire Wire Line
-	4600 4250 4750 4250
-Wire Wire Line
-	2900 4100 4100 4100
-Wire Wire Line
-	4100 4100 4100 4950
-Wire Wire Line
-	4100 4950 4750 4950
-Wire Wire Line
-	4750 5050 4000 5050
-Wire Wire Line
-	4000 5050 4000 4200
-Wire Wire Line
-	4000 4200 2900 4200
-Text HLabel 4750 4450 0    50   Output ~ 0
+Text HLabel 1250 1600 2    50   Output ~ 0
 Left_EncoderA
-Text HLabel 4750 5350 0    50   Output ~ 0
+Text HLabel 1250 2250 2    50   Output ~ 0
 Right_EncoderB
+$Comp
+L Connector:Conn_01x06_Male J13
+U 1 1 6172AE68
+P 3150 1900
+F 0 "J13" H 3258 2281 50  0000 C CNN
+F 1 "DRV8835_Right" H 3258 2190 50  0000 C CNN
+F 2 "Pin_Headers:Pin_Header_Straight_1x06_Pitch2.54mm" H 3150 1900 50  0001 C CNN
+F 3 "~" H 3150 1900 50  0001 C CNN
+	1    3150 1900
+	1    0    0    -1
+$EndComp
+$Comp
+L Connector:Conn_01x06_Male J12
+U 1 1 6172D746
+P 2650 1900
+F 0 "J12" H 2650 2300 50  0000 C CNN
+F 1 "DRV8835_Left" H 2650 2200 50  0000 C CNN
+F 2 "Pin_Headers:Pin_Header_Straight_1x06_Pitch2.54mm" H 2650 1900 50  0001 C CNN
+F 3 "~" H 2650 1900 50  0001 C CNN
+	1    2650 1900
+	-1   0    0    -1
+$EndComp
+Wire Wire Line
+	2200 1700 2450 1700
+Wire Wire Line
+	3350 1700 3650 1700
+$Comp
+L power:GND #PWR049
+U 1 1 6178417C
+P 3350 1800
+F 0 "#PWR049" H 3350 1550 50  0001 C CNN
+F 1 "GND" V 3355 1672 50  0000 R CNN
+F 2 "" H 3350 1800 50  0001 C CNN
+F 3 "" H 3350 1800 50  0001 C CNN
+	1    3350 1800
+	0    -1   -1   0
+$EndComp
+$Comp
+L power:GND #PWR048
+U 1 1 617844E4
+P 2450 2200
+F 0 "#PWR048" H 2450 1950 50  0001 C CNN
+F 1 "GND" V 2455 2072 50  0000 R CNN
+F 2 "" H 2450 2200 50  0001 C CNN
+F 3 "" H 2450 2200 50  0001 C CNN
+	1    2450 2200
+	0    1    1    0
+$EndComp
+Wire Wire Line
+	1250 1800 2450 1800
+Wire Wire Line
+	2450 1900 1250 1900
+Wire Wire Line
+	1250 2550 1900 2550
+Wire Wire Line
+	1900 2550 1900 2000
+Wire Wire Line
+	1900 2000 2450 2000
+Wire Wire Line
+	2450 2100 1950 2100
+Wire Wire Line
+	1950 2100 1950 2650
+Wire Wire Line
+	1950 2650 1250 2650
+$Comp
+L Connector:Conn_01x06_Female J5
+U 1 1 6135AD13
+P 1050 2450
+F 0 "J5" H 1078 2426 50  0000 L CNN
+F 1 "Right_Motor" H 1078 2335 50  0000 L CNN
+F 2 "Connector_JST:JST_XH_B6B-XH-AM_1x06_P2.50mm_Vertical" H 1050 2450 50  0001 C CNN
+F 3 "~" H 1050 2450 50  0001 C CNN
+	1    1050 2450
+	-1   0    0    1
+$EndComp
+$Comp
+L Connector:Conn_01x06_Female J4
+U 1 1 61359DC6
+P 1050 1700
+F 0 "J4" H 1078 1676 50  0000 L CNN
+F 1 "Left_Motor" H 1078 1585 50  0000 L CNN
+F 2 "Connector_JST:JST_XH_B6B-XH-AM_1x06_P2.50mm_Vertical" H 1050 1700 50  0001 C CNN
+F 3 "~" H 1050 1700 50  0001 C CNN
+	1    1050 1700
+	-1   0    0    1
+$EndComp
 $EndSCHEMATC

Commit message: Update schematic
Parts:
- removed J12: DRV8835_Left, Pin_Headers:Pin_Header_Straight_1x06_Pitch2.54mm, symbol Connector:Conn_01x06_Male
- removed J13: DRV8835_Right, Pin_Headers:Pin_Header_Straight_1x06_Pitch2.54mm, symbol Connector:Conn_01x06_Male
- added J8: DRV8835, Zero_Module:DRV8835Board, symbol Connector_Generic:Conn_02x06_Counter_Clockwise
Connections:
- net +3V3: now also J8.12 (Pin_12)
- net +BATT: now also J8.1 (Pin_1)
- net GND: now also J8.11 (Pin_11), J8.6 (Pin_6)
- net Left_Motor_OUT1: now also J8.10 (Pin_10)
- net Left_Motor_OUT2: now also J8.9 (Pin_9)
- net Right_Motor_OUT1: now also J8.8 (Pin_8)
- net Right_Motor_OUT2: now also J8.7 (Pin_7)
- net at J4.1 (Pin_1): now also J8.3 (Pin_3)
- net at J4.2 (Pin_2): now also J8.2 (Pin_2)
- net at J5.1 (Pin_1): now also J8.5 (Pin_5)
- net at J5.2 (Pin_2): now also J8.4 (Pin_4)
Changed lines of the file:
@@
 L power:+3.3V #PWR0104
 U 1 1 6135BC63
-P 3650 1700
-F 0 "#PWR0104" H 3650 1550 50  0001 C CNN
-F 1 "+3.3V" V 3550 1700 50  0000 C CNN
-F 2 "" H 3650 1700 50  0001 C CNN
-F 3 "" H 3650 1700 50  0001 C CNN
-	1    3650 1700
+P 3250 1700
+F 0 "#PWR0104" H 3250 1550 50  0001 C CNN
+F 1 "+3.3V" V 3150 1700 50  0000 C CNN
+F 2 "" H 3250 1700 50  0001 C CNN
+F 3 "" H 3250 1700 50  0001 C CNN
+	1    3250 1700
 	0    1    1    0
 $EndComp
@@
 	1    0    0    -1
 $EndComp
-Text HLabel 3350 1900 2    50   Input ~ 0
+Text HLabel 2950 1900 2    50   Input ~ 0
 Left_Motor_OUT1
-Text HLabel 3350 2000 2    50   Input ~ 0
+Text HLabel 2950 2000 2    50   Input ~ 0
 Left_Motor_OUT2
-Text HLabel 3350 2100 2    50   Input ~ 0
+Text HLabel 2950 2100 2    50   Input ~ 0
 Right_Motor_OUT1
-Text HLabel 3350 2200 2    50   Input ~ 0
+Text HLabel 2950 2200 2    50   Input ~ 0
 Right_Motor_OUT2
 $Comp
@@
 Text HLabel 1250 2250 2    50   Output ~ 0
 Right_EncoderB
-$Comp
-L Connector:Conn_01x06_Male J13
-U 1 1 6172AE68
-P 3150 1900
-F 0 "J13" H 3258 2281 50  0000 C CNN
-F 1 "DRV8835_Right" H 3258 2190 50  0000 C CNN
-F 2 "Pin_Headers:Pin_Header_Straight_1x06_Pitch2.54mm" H 3150 1900 50  0001 C CNN
-F 3 "~" H 3150 1900 50  0001 C CNN
-	1    3150 1900
-	1    0    0    -1
-$EndComp
-$Comp
-L Connector:Conn_01x06_Male J12
-U 1 1 6172D746
-P 2650 1900
-F 0 "J12" H 2650 2300 50  0000 C CNN
-F 1 "DRV8835_Left" H 2650 2200 50  0000 C CNN
-F 2 "Pin_Headers:Pin_Header_Straight_1x06_Pitch2.54mm" H 2650 1900 50  0001 C CNN
-F 3 "~" H 2650 1900 50  0001 C CNN
-	1    2650 1900
-	-1   0    0    -1
-$EndComp
 Wire Wire Line
 	2200 1700 2450 1700
 Wire Wire Line
-	3350 1700 3650 1700
+	2950 1700 3250 1700
 $Comp
 L power:GND #PWR049
 U 1 1 6178417C
-P 3350 1800
-F 0 "#PWR049" H 3350 1550 50  0001 C CNN
-F 1 "GND" V 3355 1672 50  0000 R CNN
-F 2 "" H 3350 1800 50  0001 C CNN
-F 3 "" H 3350 1800 50  0001 C CNN
-	1    3350 1800
+P 2950 1800
+F 0 "#PWR049" H 2950 1550 50  0001 C CNN
+F 1 "GND" V 2955 1672 50  0000 R CNN
+F 2 "" H 2950 1800 50  0001 C CNN
+F 3 "" H 2950 1800 50  0001 C CNN
+	1    2950 1800
 	0    -1   -1   0
 $EndComp
@@
 	-1   0    0    1
 $EndComp
+$Comp
+L Connector_Generic:Conn_02x06_Counter_Clockwise J8
+U 1 1 617221F1
+P 2650 1900
+F 0 "J8" H 2700 2317 50  0000 C CNN
+F 1 "DRV8835" H 2700 2226 50  0000 C CNN
+F 2 "Zero_Module:DRV8835Board" H 2650 1900 50  0001 C CNN
+F 3 "~" H 2650 1900 50  0001 C CNN
+	1    2650 1900
+	1    0    0    -1
+$EndComp
 $EndSCHEMATC

Commit message: Update
Parts:
- C13: footprint Capacitors_SMD:C_0603_HandSoldering -> Capacitors_SMD:C_0805_HandSoldering
Changed lines of the file:
@@
 F 0 "C13" H 1150 4400 50  0000 L CNN
 F 1 "22u" H 1150 4200 50  0000 L CNN
-F 2 "Capacitors_SMD:C_0603_HandSoldering" H 1138 4150 50  0001 C CNN
+F 2 "Capacitors_SMD:C_0805_HandSoldering" H 1138 4150 50  0001 C CNN
 F 3 "~" H 1100 4300 50  0001 C CNN
 	1    1100 4300

Commit message: Write about where to buy the parts
Parts:
- C12: Buy (none) -> https://akizukidenshi.com/catalog/g/gP-13374/; Vendor (none) -> https://akizukidenshi.com/catalog/g/gP-13374/
- J4, J5: Buy (none) -> https://akizukidenshi.com/catalog/g/gC-12251/; Vendor (none) -> https://akizukidenshi.com/catalog/g/gC-12251/
- J8: Buy (none) -> https://akizukidenshi.com/catalog/g/gK-09848/; Vendor (none) -> https://akizukidenshi.com/catalog/g/gK-09848/
Changed lines of the file:
@@
 F 2 "Capacitors_SMD:C_0805_HandSoldering" H 1138 4150 50  0001 C CNN
 F 3 "~" H 1100 4300 50  0001 C CNN
+F 4 "~" H 1100 4300 50  0001 C CNN "Buy"
+F 5 "~" H 1100 4300 50  0001 C CNN "Vendor"
 	1    1100 4300
 	1    0    0    -1
@@
 F 1 "0.1u" H 850 4200 50  0000 L CNN
 F 2 "Capacitors_SMD:C_0603_HandSoldering" H 838 4150 50  0001 C CNN
-F 3 "~" H 800 4300 50  0001 C CNN
+F 3 "https://akizukidenshi.com/catalog/g/gP-13374/" H 800 4300 50  0001 C CNN
+F 4 "https://akizukidenshi.com/catalog/g/gP-13374/" H 800 4300 50  0001 C CNN "Buy"
+F 5 "https://akizukidenshi.com/catalog/g/gP-13374/" H 800 4300 50  0001 C CNN "Vendor"
 	1    800  4300
 	1    0    0    -1
@@
 F 1 "Right_Motor" H 1078 2335 50  0000 L CNN
 F 2 "Connector_JST:JST_XH_B6B-XH-AM_1x06_P2.50mm_Vertical" H 1050 2450 50  0001 C CNN
-F 3 "~" H 1050 2450 50  0001 C CNN
+F 3 "https://akizukidenshi.com/catalog/g/gC-12251/" H 1050 2450 50  0001 C CNN
+F 4 "https://akizukidenshi.com/catalog/g/gC-12251/" H 1050 2450 50  0001 C CNN "Buy"
+F 5 "https://akizukidenshi.com/catalog/g/gC-12251/" H 1050 2450 50  0001 C CNN "Vendor"
 	1    1050 2450
 	-1   0    0    1
@@
 F 1 "Left_Motor" H 1078 1585 50  0000 L CNN
 F 2 "Connector_JST:JST_XH_B6B-XH-AM_1x06_P2.50mm_Vertical" H 1050 1700 50  0001 C CNN
-F 3 "~" H 1050 1700 50  0001 C CNN
+F 3 "https://akizukidenshi.com/catalog/g/gC-12251/" H 1050 1700 50  0001 C CNN
+F 4 "https://akizukidenshi.com/catalog/g/gC-12251/" H 1050 1700 50  0001 C CNN "Buy"
+F 5 "https://akizukidenshi.com/catalog/g/gC-12251/" H 1050 1700 50  0001 C CNN "Vendor"
 	1    1050 1700
 	-1   0    0    1
@@
 F 1 "DRV8835" H 2700 2226 50  0000 C CNN
 F 2 "Zero_Module:DRV8835Board" H 2650 1900 50  0001 C CNN
-F 3 "~" H 2650 1900 50  0001 C CNN
+F 3 "https://akizukidenshi.com/catalog/g/gK-09848/" H 2650 1900 50  0001 C CNN
+F 4 "https://akizukidenshi.com/catalog/g/gK-09848/" H 2650 1900 50  0001 C CNN "Buy"
+F 5 "https://akizukidenshi.com/catalog/g/gK-09848/" H 2650 1900 50  0001 C CNN "Vendor"
 	1    2650 1900
 	1    0    0    -1
