File: pcb/power.sch (KiCad schematic (older format))
At the start: 18 parts, among them J1 BATTERY1, J2 BATTERY2, J3 VX07803-500, Q1 IRLML6402, SW1 POWER_SWITCH, U1 NJU77701F

Commit message: Make netlist
Parts:
- C1, C2, C3: footprint (none) -> Capacitors_SMD:C_0603_HandSoldering
- D1: footprint (none) -> LEDs:LED_0603_HandSoldering
- J1, J2: footprint (none) -> Connectors_Molex:Molex_PicoBlade_53047-0210_02x1.25mm_Straight; symbol Connector:Conn_01x02_Male -> Connector:Conn_01x02_Female
- J3, SW1: footprint (none) -> Pin_Headers:Pin_Header_Straight_1x03_Pitch2.54mm
- L1: value 100u -> 10u; footprint (none) -> Resistors_SMD:R_1210_HandSoldering
- Q1: footprint Package_TO_SOT_SMD:SOT-23 -> TO_SOT_Packages_SMD:SOT-23
- R1, R2, R3, R4, R5, R6, R7: footprint (none) -> Resistors_SMD:R_0603_HandSoldering
- U1: footprint Package_TO_SOT_SMD:SOT-23-5 -> TO_SOT_Packages_SMD:SOT-23-5_HandSoldering
Connections:
- net GND: now also J2.2 (Pin_2); no longer J2.1 (Pin_1)
- net at Q1.2 (S), R1.1: now also J1.1 (Pin_1); no longer J1.2 (Pin_2)
- new net: J1.2 (Pin_2), J2.1 (Pin_1)
Changed lines of the file:
@@
 F 0 "Q1" V 3192 3000 50  0000 C CNN
 F 1 "IRLML6402" V 3101 3000 50  0000 C CNN
-F 2 "Package_TO_SOT_SMD:SOT-23" H 3050 2925 50  0001 L CIN
+F 2 "TO_SOT_Packages_SMD:SOT-23" H 3050 2925 50  0001 L CIN
 F 3 "https://www.infineon.com/dgdl/irlml6402pbf.pdf?fileId=5546d462533600a401535668d5c2263c" H 2850 3000 50  0001 L CNN
 	1    2850 3000
@@
 F 0 "R1" V 2793 3400 50  0000 C CNN
 F 1 "10k" V 3000 3400 50  0000 C CNN
-F 2 "" V 2930 3400 50  0001 C CNN
+F 2 "Resistors_SMD:R_0603_HandSoldering" V 2930 3400 50  0001 C CNN
 F 3 "~" H 3000 3400 50  0001 C CNN
 	1    3000 3400
@@
 	2850 3200 2850 3400
 $Comp
-L Connector:Conn_01x02_Male J1
+L Connector:Conn_01x02_Female J1
 U 1 1 612C4678
-P 3350 2700
-F 0 "J1" V 3412 2744 50  0000 L CNN
-F 1 "BATTERY1" V 3503 2744 50  0000 L CNN
-F 2 "" H 3350 2700 50  0001 C CNN
-F 3 "~" H 3350 2700 50  0001 C CNN
-	1    3350 2700
-	0    1    1    0
+P 3250 2700
+F 0 "J1" V 3312 2744 50  0000 L CNN
+F 1 "BATTERY1" V 3403 2744 50  0000 L CNN
+F 2 "Connectors_Molex:Molex_PicoBlade_53047-0210_02x1.25mm_Straight" H 3250 2700 50  0001 C CNN
+F 3 "~" H 3250 2700 50  0001 C CNN
+	1    3250 2700
+	0    -1   -1   0
 $EndComp
 Wire Wire Line
@@
 	3350 2900 4000 2900
 $Comp
-L Connector:Conn_01x02_Male J2
+L Connector:Conn_01x02_Female J2
 U 1 1 612C59BF
-P 4100 2700
-F 0 "J2" V 4162 2744 50  0000 L CNN
-F 1 "BATTERY2" V 4253 2744 50  0000 L CNN
-F 2 "" H 4100 2700 50  0001 C CNN
-F 3 "~" H 4100 2700 50  0001 C CNN
-	1    4100 2700
-	0    1    1    0
+P 4000 2700
+F 0 "J2" V 4062 2744 50  0000 L CNN
+F 1 "BATTERY2" V 4153 2744 50  0000 L CNN
+F 2 "Connectors_Molex:Molex_PicoBlade_53047-0210_02x1.25mm_Straight" H 4000 2700 50  0001 C CNN
+F 3 "~" H 4000 2700 50  0001 C CNN
+	1    4000 2700
+	0    -1   -1   0
 $EndComp
 Wire Wire Line
@@
 F 0 "SW1" V 2804 3898 50  0000 L CNN
 F 1 "POWER_SWITCH" V 2895 3898 50  0000 L CNN
-F 2 "" H 2850 3750 50  0001 C CNN
+F 2 "Pin_Headers:Pin_Header_Straight_1x03_Pitch2.54mm" H 2850 3750 50  0001 C CNN
 F 3 "~" H 2850 3750 50  0001 C CNN
 	1    2850 3750
@@
 F 0 "R5" H 4920 3696 50  0000 L CNN
 F 1 "10k" V 4850 3600 50  0000 L CNN
-F 2 "" V 4780 3650 50  0001 C CNN
+F 2 "Resistors_SMD:R_0603_HandSoldering" V 4780 3650 50  0001 C CNN
 F 3 "~" H 4850 3650 50  0001 C CNN
 	1    4850 3650
@@
 F 0 "C2" H 5465 3696 50  0000 L CNN
 F 1 "0.1u" H 5465 3605 50  0000 L CNN
-F 2 "" H 5388 3500 50  0001 C CNN
+F 2 "Capacitors_SMD:C_0603_HandSoldering" H 5388 3500 50  0001 C CNN
 F 3 "~" H 5350 3650 50  0001 C CNN
 	1    5350 3650
@@
 F 0 "U1" H 6400 3500 50  0000 L CNN
 F 1 "NJU77701F" H 6250 3250 50  0000 L CNN
-F 2 "Package_TO_SOT_SMD:SOT-23-5" H 6200 3200 50  0001 L CNN
+F 2 "TO_SOT_Packages_SMD:SOT-23-5_HandSoldering" H 6200 3200 50  0001 L CNN
 F 3 "http://www.ti.com/lit/ds/symlink/lmh6609.pdf" H 6300 3600 50  0001 C CNN
 	1    6300 3400
@@
 F 0 "J3" H 2042 4275 50  0000 C CNN
 F 1 "VX07803-500" H 2042 4366 50  0000 C CNN
-F 2 "" H 2150 4600 50  0001 C CNN
+F 2 "Pin_Headers:Pin_Header_Straight_1x03_Pitch2.54mm" H 2150 4600 50  0001 C CNN
 F 3 "~" H 2150 4600 50  0001 C CNN
 	1    2150 4600
@@
 F 0 "R2" H 4020 4546 50  0000 L CNN
 F 1 "1k" V 3950 4450 50  0000 L CNN
-F 2 "" V 3880 4500 50  0001 C CNN
+F 2 "Resistors_SMD:R_0603_HandSoldering" V 3880 4500 50  0001 C CNN
 F 3 "~" H 3950 4500 50  0001 C CNN
 	1    3950 4500
@@
 F 0 "D1" V 3989 4682 50  0000 R CNN
 F 1 "PWR_LED" V 3898 4682 50  0000 R CNN
-F 2 "" H 3950 4800 50  0001 C CNN
+F 2 "LEDs:LED_0603_HandSoldering" H 3950 4800 50  0001 C CNN
 F 3 "~" H 3950 4800 50  0001 C CNN
 	1    3950 4800
@@
 P 5000 4500
 F 0 "L1" V 5100 4450 50  0000 L CNN
-F 1 "100u" V 4950 4400 50  0000 L CNN
-F 2 "" H 5000 4500 50  0001 C CNN
+F 1 "10u" V 4950 4400 50  0000 L CNN
+F 2 "Resistors_SMD:R_1210_HandSoldering" H 5000 4500 50  0001 C CNN
 F 3 "~" H 5000 4500 50  0001 C CNN
 	1    5000 4500
@@
 F 0 "C1" H 5265 4846 50  0000 L CNN
 F 1 "0.1u" H 5265 4755 50  0000 L CNN
-F 2 "" H 5188 4650 50  0001 C CNN
+F 2 "Capacitors_SMD:C_0603_HandSoldering" H 5188 4650 50  0001 C CNN
 F 3 "~" H 5150 4800 50  0001 C CNN
 	1    5150 4800
@@
 F 0 "R3" V 4600 4500 50  0000 C CNN
 F 1 "10" V 4700 4500 50  0000 C CNN
-F 2 "" V 4630 4500 50  0001 C CNN
+F 2 "Resistors_SMD:R_0603_HandSoldering" V 4630 4500 50  0001 C CNN
 F 3 "~" H 4700 4500 50  0001 C CNN
 	1    4700 4500
@@
 F 0 "R6" V 5550 4650 50  0000 C CNN
 F 1 "1k" V 5650 4650 50  0000 C CNN
-F 2 "" V 5580 4650 50  0001 C CNN
+F 2 "Resistors_SMD:R_0603_HandSoldering" V 5580 4650 50  0001 C CNN
 F 3 "~" H 5650 4650 50  0001 C CNN
 	1    5650 4650
@@
 F 0 "R7" V 5550 4950 50  0000 C CNN
 F 1 "1k" V 5650 4950 50  0000 C CNN
-F 2 "" V 5580 4950 50  0001 C CNN
+F 2 "Resistors_SMD:R_0603_HandSoldering" V 5580 4950 50  0001 C CNN
 F 3 "~" H 5650 4950 50  0001 C CNN
 	1    5650 4950
@@
 F 0 "C3" H 6015 4996 50  0000 L CNN
 F 1 "0.1u" H 6015 4905 50  0000 L CNN
-F 2 "" H 5938 4800 50  0001 C CNN
+F 2 "Capacitors_SMD:C_0603_HandSoldering" H 5938 4800 50  0001 C CNN
 F 3 "~" H 5900 4950 50  0001 C CNN
 	1    5900 4950
@@
 F 0 "R4" H 4920 3046 50  0000 L CNN
 F 1 "20k" V 4850 2950 50  0000 L CNN
-F 2 "" V 4780 3000 50  0001 C CNN
+F 2 "Resistors_SMD:R_0603_HandSoldering" V 4780 3000 50  0001 C CNN
 F 3 "~" H 4850 3000 50  0001 C CNN
 	1    4850 3000

Commit message: Update pcb
Parts:
- added C14, C15: 0.1u, Capacitors_SMD:C_0603_HandSoldering, symbol Device:C
- added C16, C17: 10u, Capacitors_SMD:C_0603_HandSoldering, symbol Device:C
- added C18: 2.2u, Capacitors_SMD:C_0603_HandSoldering, symbol Device:C
- added J12: GND_PIN, Pin_Headers:Pin_Header_Straight_1x01_Pitch2.54mm, symbol Connector:Conn_01x01_Female
- added J9: BATT_PIN, Pin_Headers:Pin_Header_Straight_1x01_Pitch2.54mm, symbol Connector:Conn_01x01_Female
Connections:
- net +3.3VA: now also C18.1
- net +3V3: now also C15.1, C17.1
- net +BATT: now also C14.1, C16.1
- net GND: now also C14.2, C15.2, C16.2, C17.2, C18.2, J12.1 (Pin_1)
- net at J1.1 (Pin_1), Q1.2 (S), R1.1: now also J9.1 (Pin_1)

Commit message: Write about where to buy the parts
Parts:
- C1, C14, C15, C2, C3: Buy (none) -> https://akizukidenshi.com/catalog/g/gP-13374/; Vendor (none) -> https://akizukidenshi.com/catalog/g/gP-13374/
- C16, C17: Buy (none) -> https://akizukidenshi.com/catalog/g/gP-13161/; Vendor (none) -> https://akizukidenshi.com/catalog/g/gP-13161/
- C18: Buy (none) -> https://akizukidenshi.com/catalog/g/gP-16077/; Vendor (none) -> https://akizukidenshi.com/catalog/g/gP-16077/
- D1: Buy (none) -> https://akizukidenshi.com/catalog/g/gI-11879/; Vendor (none) -> https://akizukidenshi.com/catalog/g/gI-11879/
- J1, J2: Buy (none) -> https://www.sengoku.co.jp/mod/sgk_cart/detail.php?code=EEHD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; Vendor (none) -> https://www.sengoku.co.jp/mod/sgk_cart/detail.php?code=EEHD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
- J3: Buy (none) -> https://akizukidenshi.com/catalog/g/gM-15148/; Vendor (none) -> https://akizukidenshi.com/catalog/g/gM-15148/
- L1: Buy (none) -> https://akizukidenshi.com/catalog/g/gP-14978/; Vendor (none) -> https://akizukidenshi.com/catalog/g/gP-14978/
- Q1: Buy (none) -> https://www.infineon.com/dgdl/irlml6402pbf.pdf?fileId=5546d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; Vendor (none) -> https://www.infineon.com/dgdl/irlml6402pbf.pdf?fileId=5546d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
- R2, R6, R7: Buy (none) -> https://akizukidenshi.com/catalog/g/gR-14122/; Vendor (none) -> https://akizukidenshi.com/catalog/g/gR-14122/
- U1: Buy (none) -> https://akizukidenshi.com/catalog/g/gI-07103/; Vendor (none) -> https://akizukidenshi.com/catalog/g/gI-07103/
Changed lines of the file:
@@
 F 2 "TO_SOT_Packages_SMD:SOT-23" H 3050 2925 50  0001 L CIN
 F 3 "https://www.infineon.com/dgdl/irlml6402pbf.pdf?fileId=5546d462533600a401535668d5c2263c" H 2850 3000 50  0001 L CNN
+F 4 "https://www.infineon.com/dgdl/irlml6402pbf.pdf?fileId=5546d462533600a401535668d5c2263c" H 2850 3000 50  0001 C CNN "Buy"
+F 5 "https://www.infineon.com/dgdl/irlml6402pbf.pdf?fileId=5546d462533600a401535668d5c2263c" H 2850 3000 50  0001 C CNN "Vendor"
 	1    2850 3000
 	0    -1   -1   0
@@
 F 2 "Resistors_SMD:R_0603_HandSoldering" V 2930 3400 50  0001 C CNN
 F 3 "~" H 3000 3400 50  0001 C CNN
+F 4 "~" H 3000 3400 50  0001 C CNN "Buy"
+F 5 "~" H 3000 3400 50  0001 C CNN "Vendor"
 	1    3000 3400
 	0    1    1    0
@@
 F 1 "BATTERY1" V 3403 2744 50  0000 L CNN
 F 2 "Connectors_Molex:Molex_PicoBlade_53047-0210_02x1.25mm_Straight" H 3250 2700 50  0001 C CNN
-F 3 "~" H 3250 2700 50  0001 C CNN
+F 3 "https://www.sengoku.co.jp/mod/sgk_cart/detail.php?code=EEHD-4B5T" H 3250 2700 50  0001 C CNN
+F 4 "https://www.sengoku.co.jp/mod/sgk_cart/detail.php?code=EEHD-4B5T" H 3250 2700 50  0001 C CNN "Buy"
+F 5 "https://www.sengoku.co.jp/mod/sgk_cart/detail.php?code=EEHD-4B5T" H 3250 2700 50  0001 C CNN "Vendor"
 	1    3250 2700
 	0    -1   -1   0
@@
 F 1 "BATTERY2" V 4153 2744 50  0000 L CNN
 F 2 "Connectors_Molex:Molex_PicoBlade_53047-0210_02x1.25mm_Straight" H 4000 2700 50  0001 C CNN
-F 3 "~" H 4000 2700 50  0001 C CNN
+F 3 "https://www.sengoku.co.jp/mod/sgk_cart/detail.php?code=EEHD-4B5T" H 4000 2700 50  0001 C CNN
+F 4 "https://www.sengoku.co.jp/mod/sgk_cart/detail.php?code=EEHD-4B5T" H 4000 2700 50  0001 C CNN "Buy"
+F 5 "https://www.sengoku.co.jp/mod/sgk_cart/detail.php?code=EEHD-4B5T" H 4000 2700 50  0001 C CNN "Vendor"
 	1    4000 2700
 	0    -1   -1   0
@@
 F 2 "Pin_Headers:Pin_Header_Straight_1x03_Pitch2.54mm" H 2850 3750 50  0001 C CNN
 F 3 "~" H 2850 3750 50  0001 C CNN
+F 4 "~" H 2850 3750 50  0001 C CNN "Buy"
+F 5 "~" H 2850 3750 50  0001 C CNN "Vendor"
 	1    2850 3750
 	0    1    1    0
@@
 F 2 "Resistors_SMD:R_0603_HandSoldering" V 4780 3650 50  0001 C CNN
 F 3 "~" H 4850 3650 50  0001 C CNN
+F 4 "~" H 4850 3650 50  0001 C CNN "Buy"
+F 5 "~" H 4850 3650 50  0001 C CNN "Vendor"
 	1    4850 3650
 	1    0    0    -1
@@
 F 1 "0.1u" H 5465 3605 50  0000 L CNN
 F 2 "Capacitors_SMD:C_0603_HandSoldering" H 5388 3500 50  0001 C CNN
-F 3 "~" H 5350 3650 50  0001 C CNN
+F 3 "https://akizukidenshi.com/catalog/g/gP-13374/" H 5350 3650 50  0001 C CNN
+F 4 "https://akizukidenshi.com/catalog/g/gP-13374/" H 5350 3650 50  0001 C CNN "Buy"
+F 5 "https://akizukidenshi.com/catalog/g/gP-13374/" H 5350 3650 50  0001 C CNN "Vendor"
 	1    5350 3650
 	1    0    0    -1
@@
 F 1 "NJU77701F" H 6250 3250 50  0000 L CNN
 F 2 "TO_SOT_Packages_SMD:SOT-23-5_HandSoldering" H 6200 3200 50  0001 L CNN
-F 3 "http://www.ti.com/lit/ds/symlink/lmh6609.pdf" H 6300 3600 50  0001 C CNN
+F 3 "https://akizukidenshi.com/catalog/g/gI-07103/" H 6300 3600 50  0001 C CNN
+F 4 "https://akizukidenshi.com/catalog/g/gI-07103/" H 6300 3400 50  0001 C CNN "Buy"
+F 5 "https://akizukidenshi.com/catalog/g/gI-07103/" H 6300 3400 50  0001 C CNN "Vendor"
 	1    6300 3400
 	1    0    0    -1
@@
 F 1 "1k" V 3950 4450 50  0000 L CNN
 F 2 "Resistors_SMD:R_0603_HandSoldering" V 3880 4500 50  0001 C CNN
-F 3 "~" H 3950 4500 50  0001 C CNN
+F 3 "https://akizukidenshi.com/catalog/g/gR-14122/" H 3950 4500 50  0001 C CNN
+F 4 "https://akizukidenshi.com/catalog/g/gR-14122/" H 3950 4500 50  0001 C CNN "Buy"
+F 5 "https://akizukidenshi.com/catalog/g/gR-14122/" H 3950 4500 50  0001 C CNN "Vendor"
 	1    3950 4500
 	1    0    0    -1
@@
 F 1 "PWR_LED" V 3898 4682 50  0000 R CNN
 F 2 "LEDs:LED_0603_HandSoldering" H 3950 4800 50  0001 C CNN
-F 3 "~" H 3950 4800 50  0001 C CNN
+F 3 "https://akizukidenshi.com/catalog/g/gI-11879/" H 3950 4800 50  0001 C CNN
+F 4 "https://akizukidenshi.com/catalog/g/gI-11879/" H 3950 4800 50  0001 C CNN "Buy"
+F 5 "https://akizukidenshi.com/catalog/g/gI-11879/" H 3950 4800 50  0001 C CNN "Vendor"
 	1    3950 4800
 	0    -1   -1   0
@@
 F 1 "10u" V 4950 4400 50  0000 L CNN
 F 2 "Resistors_SMD:R_1210_HandSoldering" H 5000 4500 50  0001 C CNN
-F 3 "~" H 5000 4500 50  0001 C CNN
+F 3 "https://akizukidenshi.com/catalog/g/gP-14978/" H 5000 4500 50  0001 C CNN
+F 4 "https://akizukidenshi.com/catalog/g/gP-14978/" H 5000 4500 50  0001 C CNN "Buy"
+F 5 "https://akizukidenshi.com/catalog/g/gP-14978/" H 5000 4500 50  0001 C CNN "Vendor"
 	1    5000 4500
 	0    -1   -1   0
@@
 F 1 "0.1u" H 5265 4755 50  0000 L CNN
 F 2 "Capacitors_SMD:C_0603_HandSoldering" H 5188 4650 50  0001 C CNN
-F 3 "~" H 5150 4800 50  0001 C CNN
+F 3 "https://akizukidenshi.com/catalog/g/gP-13374/" H 5150 4800 50  0001 C CNN
+F 4 "https://akizukidenshi.com/catalog/g/gP-13374/" H 5150 4800 50  0001 C CNN "Buy"
+F 5 "https://akizukidenshi.com/catalog/g/gP-13374/" H 5150 4800 50  0001 C CNN "Vendor"
 	1    5150 4800
 	1    0    0    -1
@@
 F 2 "Resistors_SMD:R_0603_HandSoldering" V 4630 4500 50  0001 C CNN
 F 3 "~" H 4700 4500 50  0001 C CNN
+F 4 "~" H 4700 4500 50  0001 C CNN "Buy"
+F 5 "~" H 4700 4500 50  0001 C CNN "Vendor"
 	1    4700 4500
 	0    1    1    0
@@
 F 1 "1k" V 5650 4650 50  0000 C CNN
 F 2 "Resistors_SMD:R_0603_HandSoldering" V 5580 4650 50  0001 C CNN
-F 3 "~" H 5650 4650 50  0001 C CNN
+F 3 "https://akizukidenshi.com/catalog/g/gR-14122/" H 5650 4650 50  0001 C CNN
+F 4 "https://akizukidenshi.com/catalog/g/gR-14122/" H 5650 4650 50  0001 C CNN "Buy"
+F 5 "https://akizukidenshi.com/catalog/g/gR-14122/" H 5650 4650 50  0001 C CNN "Vendor"
 	1    5650 4650
 	-1   0    0    1
@@
 F 1 "1k" V 5650 4950 50  0000 C CNN
 F 2 "Resistors_SMD:R_0603_HandSoldering" V 5580 4950 50  0001 C CNN
-F 3 "~" H 5650 4950 50  0001 C CNN
+F 3 "https://akizukidenshi.com/catalog/g/gR-14122/" H 5650 4950 50  0001 C CNN
+F 4 "https://akizukidenshi.com/catalog/g/gR-14122/" H 5650 4950 50  0001 C CNN "Buy"
+F 5 "https://akizukidenshi.com/catalog/g/gR-14122/" H 5650 4950 50  0001 C CNN "Vendor"
 	1    5650 4950
 	-1   0    0    1
@@
 F 1 "0.1u" H 6015 4905 50  0000 L CNN
 F 2 "Capacitors_SMD:C_0603_HandSoldering" H 5938 4800 50  0001 C CNN
-F 3 "~" H 5900 4950 50  0001 C CNN
+F 3 "https://akizukidenshi.com/catalog/g/gP-13374/" H 5900 4950 50  0001 C CNN
+F 4 "https://akizukidenshi.com/catalog/g/gP-13374/" H 5900 4950 50  0001 C CNN "Buy"
+F 5 "https://akizukidenshi.com/catalog/g/gP-13374/" H 5900 4950 50  0001 C CNN "Vendor"
 	1    5900 4950
 	1    0    0    -1
@@
 F 2 "Resistors_SMD:R_0603_HandSoldering" V 4780 3000 50  0001 C CNN
 F 3 "~" H 4850 3000 50  0001 C CNN
+F 4 "~" H 4850 3000 50  0001 C CNN "Buy"
+F 5 "~" H 4850 3000 50  0001 C CNN "Vendor"
 	1    4850 3000
 	1    0    0    -1
@@
 F 1 "VX07803-500" H 2042 4366 50  0000 C CNN
 F 2 "Pin_Headers:Pin_Header_Straight_1x03_Pitch2.54mm" H 2150 4600 50  0001 C CNN
-F 3 "~" H 2150 4600 50  0001 C CNN
+F 3 "https://akizukidenshi.com/catalog/g/gM-15148/" H 2150 4600 50  0001 C CNN
+F 4 "https://akizukidenshi.com/catalog/g/gM-15148/" H 2150 4600 50  0001 C CNN "Buy"
+F 5 "https://akizukidenshi.com/catalog/g/gM-15148/" H 2150 4600 50  0001 C CNN "Vendor"
 	1    2150 4600
 	-1   0    0    1
@@
 F 2 "Pin_Headers:Pin_Header_Straight_1x01_Pitch2.54mm" H 3800 3350 50  0001 C CNN
 F 3 "~" H 3800 3350 50  0001 C CNN
+F 4 "~" H 3800 3350 50  0001 C CNN "Buy"
+F 5 "~" H 3800 3350 50  0001 C CNN "Vendor"
 	1    3800 3350
 	0    1    1    0
@@
 F 2 "Pin_Headers:Pin_Header_Straight_1x01_Pitch2.54mm" H 3450 3350 50  0001 C CNN
 F 3 "~" H 3450 3350 50  0001 C CNN
+F 4 "~" H 3450 3350 50  0001 C CNN "Buy"
+F 5 "~" H 3450 3350 50  0001 C CNN "Vendor"
 	1    3450 3350
 	0    1    1    0
@@
 F 1 "0.1u" H 815 4905 50  0000 L CNN
 F 2 "Capacitors_SMD:C_0603_HandSoldering" H 738 4800 50  0001 C CNN
-F 3 "~" H 700 4950 50  0001 C CNN
+F 3 "https://akizukidenshi.com/catalog/g/gP-13374/" H 700 4950 50  0001 C CNN
+F 4 "https://akizukidenshi.com/catalog/g/gP-13374/" H 700 4950 50  0001 C CNN "Buy"
+F 5 "https://akizukidenshi.com/catalog/g/gP-13374/" H 700 4950 50  0001 C CNN "Vendor"
 	1    700  4950
 	1    0    0    -1
@@
 F 1 "10u" H 1215 4905 50  0000 L CNN
 F 2 "Capacitors_SMD:C_0603_HandSoldering" H 1138 4800 50  0001 C CNN
-F 3 "~" H 1100 4950 50  0001 C CNN
+F 3 "https://akizukidenshi.com/catalog/g/gP-13161/" H 1100 4950 50  0001 C CNN
+F 4 "https://akizukidenshi.com/catalog/g/gP-13161/" H 1100 4950 50  0001 C CNN "Buy"
+F 5 "https://akizukidenshi.com/catalog/g/gP-13161/" H 1100 4950 50  0001 C CNN "Vendor"
 	1    1100 4950
 	1    0    0    -1
@@
 F 1 "0.1u" H 815 5805 50  0000 L CNN
 F 2 "Capacitors_SMD:C_0603_HandSoldering" H 738 5700 50  0001 C CNN
-F 3 "~" H 700 5850 50  0001 C CNN
+F 3 "https://akizukidenshi.com/catalog/g/gP-13374/" H 700 5850 50  0001 C CNN
+F 4 "https://akizukidenshi.com/catalog/g/gP-13374/" H 700 5850 50  0001 C CNN "Buy"
+F 5 "https://akizukidenshi.com/catalog/g/gP-13374/" H 700 5850 50  0001 C CNN "Vendor"
 	1    700  5850
 	1    0    0    -1
@@
 F 1 "10u" H 1215 5805 50  0000 L CNN
 F 2 "Capacitors_SMD:C_0603_HandSoldering" H 1138 5700 50  0001 C CNN
-F 3 "~" H 1100 5850 50  0001 C CNN
+F 3 "https://akizukidenshi.com/catalog/g/gP-13161/" H 1100 5850 50  0001 C CNN
+F 4 "https://akizukidenshi.com/catalog/g/gP-13161/" H 1100 5850 50  0001 C CNN "Buy"
+F 5 "https://akizukidenshi.com/catalog/g/gP-13161/" H 1100 5850 50  0001 C CNN "Vendor"
 	1    1100 5850
 	1    0    0    -1
@@
 F 1 "2.2u" H 815 6555 50  0000 L CNN
 F 2 "Capacitors_SMD:C_0603_HandSoldering" H 738 6450 50  0001 C CNN
-F 3 "~" H 700 6600 50  0001 C CNN
+F 3 "https://akizukidenshi.com/catalog/g/gP-16077/" H 700 6600 50  0001 C CNN
+F 4 "https://akizukidenshi.com/catalog/g/gP-16077/" H 700 6600 50  0001 C CNN "Buy"
+F 5 "https://akizukidenshi.com/catalog/g/gP-16077/" H 700 6600 50  0001 C CNN "Vendor"
 	1    700  6600
 	1    0    0    -1
